Commit message: add new ramps

File: definitions/moon_terrain/model.xacro (robot description, xacro)
@@ -1,5 +1,5 @@
 <?xml version="1.0" ?>
 <sdf version="1.5" xmlns:xacro="http://www.ros.org/wiki/xacro">
-  <model name="rover_amalia_turret">
+  <model name="moon_terrain">
     <static>true</static>
     <link name="link">

File: definitions/ramp-single-low/model.xacro (robot description, xacro)
@@ -2,6 +2,6 @@
 <sdf version="1.5" xmlns:xacro="http://www.ros.org/wiki/xacro">
   <xacro:include filename="./ramp1.xacro" />
-  <model name="ramp1">
-    <xacro:ramp1 sx="0.5" sy="0.5" sz="0.4"/>
+  <model name="ramp-single-low">
+    <xacro:ramp1 ox="0" oy="0" oz="0" rx="0" ry="0" rz="0" sx="0.5" sy="0.5" sz="0.4" suffix=''/>
     <pose>0 0 0 0 0 0</pose>
   </model>

File: definitions/ramp-single-low/ramp1.xacro (robot description, xacro)
@@ -2,24 +2,26 @@
 <robot name="ramp1" xmlns:xacro="http://www.ros.org/wiki/xacro">
   <xacro:property name="pi" value="3.1415926" />
-  <xacro:macro name="ramp1" params="sx sy sz">
-    <link name="ramp1_link">
+  <xacro:macro name="ramp1" params="ox oy oz rx ry rz sx sy sz suffix">
+    <link name="ramp1_link_${suffix}">
+        <pose>${ox} ${oy} ${oz} ${rx} ${ry} ${rz}</pose>
       <inertial>
-        <pose>0 0 0 0 0 0</pose>
-        <mass>100</mass>
+        <!--<pose>${ox} ${oy} ${oz} ${rx} ${ry} ${rz}</pose>-->
+        <pose>${rx/5*rz} 0 0 0 0 0</pose>
+        <mass>1000</mass>
       </inertial>
-      <collision name="ramp1_collision">
+      <collision name="ramp1_collision_${suffix}">
         <pose>0 0 0 0 0 0</pose>
         <geometry>
           <mesh>
-            <uri>model://ramp1/meshes/ramp1.dae</uri>
+            <uri>model://ramp-single-low/meshes/ramp1.dae</uri>
             <scale>${sx} ${sy} ${sz}</scale>
           </mesh>
         </geometry>
       </collision>
-      <visual name="ramp1_visual">
+      <visual name="ramp1_visual_${suffix}">
         <pose>0 0 0 0 0 0</pose>
         <geometry>
           <mesh>
-            <uri>model://ramp1/meshes/ramp1.dae</uri>
+            <uri>model://ramp-single-low/meshes/ramp1.dae</uri>
             <scale>${sx} ${sy} ${sz}</scale>
           </mesh>
