Commit message: setup new directories for xacro

File: definitions/rover_amalia/model.xacro (robot description, xacro)
@@ -1,6 +1,6 @@
-<?xml version="1.0"?>
+<?xml version="1.0" ?>
 <sdf version="1.5">
-  <model name='rover_amalia'>
-    <plugin name="skid_steer_drive" filename="libgazebo_ros_skid_steer_drive.so">
+  <model name="rover_amalia">
+    <plugin filename="libgazebo_ros_skid_steer_drive.so" name="skid_steer_drive">
       <robotNamespace>rover_amalia</robotNamespace>
       <broadcastTF>1</broadcastTF>
@@ -19,5 +19,5 @@
     </plugin>
     <static>0</static>
-    <link name='chassis'>
+    <link name="chassis">
       <pose>0 0 0 0 0 0</pose>
       <inertial>
@@ -33,5 +33,5 @@
         </inertia>
       </inertial>
-      <collision name='chassis_collision'>
+      <collision name="chassis_collision">
         <pose>0 0 0 0 -0 0</pose>
         <geometry>
@@ -43,13 +43,13 @@
         <surface>
           <contact>
-            <ode />
-          </contact>
-          <bounce />
-          <friction>
-            <ode />
-          </friction>
-        </surface>
-      </collision>
-      <collision name='chassis_collision_base'>
+            <ode/>
+          </contact>
+          <bounce/>
+          <friction>
+            <ode/>
+          </friction>
+        </surface>
+      </collision>
+      <collision name="chassis_collision_base">
         <pose>0.195 0 0.073 0 -0 0</pose>
         <geometry>
@@ -61,13 +61,13 @@
         <surface>
           <contact>
-            <ode />
-          </contact>
-          <bounce />
-          <friction>
-            <ode />
-          </friction>
-        </surface>
-      </collision>
-      <collision name='chassis_collision_leg_f_l'>
+            <ode/>
+          </contact>
+          <bounce/>
+          <friction>
+            <ode/>
+          </friction>
+        </surface>
+      </collision>
+      <collision name="chassis_collision_leg_f_l">
         <pose>0.177943 0.19 -0.0987583 0 -0.5 0</pose>
         <geometry>
@@ -80,13 +80,13 @@
         <surface>
           <contact>
-            <ode />
-          </contact>
-          <bounce />
-          <friction>
-            <ode />
-          </friction>
-        </surface>
-      </collision>
-      <collision name='chassis_collision_leg_f_r'>
+            <ode/>
+          </contact>
+          <bounce/>
+          <friction>
+            <ode/>
+          </friction>
+        </surface>
+      </collision>
+      <collision name="chassis_collision_leg_f_r">
         <pose>0.177943 -0.19 -0.0987583 0 -0.5 0</pose>
         <geometry>
@@ -99,13 +99,13 @@
         <surface>
           <contact>
-            <ode />
-          </contact>
-          <bounce />
-          <friction>
-            <ode />
-          </friction>
-        </surface>
-      </collision>
-      <collision name='chassis_collision_leg_p_l'>
+            <ode/>
+          </contact>
+          <bounce/>
+          <friction>
+            <ode/>
+          </friction>
+        </surface>
+      </collision>
+      <collision name="chassis_collision_leg_p_l">
         <pose>-0.177943 0.19 -0.0987583 0 0.5 0</pose>
         <geometry>
@@ -118,13 +118,13 @@
         <surface>
           <contact>
-            <ode />
-          </contact>
-          <bounce />
-          <friction>
-            <ode />
-          </friction>
-        </surface>
-      </collision>
-      <collision name='chassis_collision_leg_p_r'>
+            <ode/>
+          </contact>
+          <bounce/>
+          <friction>
+            <ode/>
+          </friction>
+        </surface>
+      </collision>
+      <collision name="chassis_collision_leg_p_r">
         <pose>-0.177943 -0.19 -0.0987583 0 0.5 0</pose>
         <geometry>
@@ -137,13 +137,13 @@
         <surface>
           <contact>
-            <ode />
-          </contact>
-          <bounce />
-          <friction>
-            <ode />
-          </friction>
-        </surface>
-      </collision>
-      <visual name='chassis_visual'>
+            <ode/>
+          </contact>
+          <bounce/>
+          <friction>
+            <ode/>
+          </friction>
+        </surface>
+      </collision>
+      <visual name="chassis_visual">
         <pose>0 0 0 0 -0 0</pose>
         <geometry>
@@ -153,5 +153,5 @@
         </geometry>
       </visual>
-      <visual name='chassis_visual_Range_Front'>
+      <visual name="chassis_visual_Range_Front">
         <pose>0.246 0 -0.05 0 -0 0</pose>
         <geometry>
@@ -161,5 +161,5 @@
         </geometry>
       </visual>
-      <visual name='chassis_visual_Range_Front_Down'>
+      <visual name="chassis_visual_Range_Front_Down">
         <pose>0.246 0 -0.05 0 1.57 0</pose>
         <geometry>
@@ -169,5 +169,5 @@
         </geometry>
       </visual>
-      <visual name='chassis_visual_Range_Post'>
+      <visual name="chassis_visual_Range_Post">
         <pose>-0.246 0 -0.05 3.14159 0.00159265 3.14159</pose>
         <geometry>
@@ -177,5 +177,5 @@
         </geometry>
       </visual>
-      <visual name='chassis_visual_Range_Post_Down'>
+      <visual name="chassis_visual_Range_Post_Down">
         <pose>-0.246 0 -0.05 0 1.57 0</pose>
         <geometry>
@@ -185,5 +185,5 @@
         </geometry>
       </visual>
-      <visual name='chassis_visual_base'>
+      <visual name="chassis_visual_base">
         <pose>0.195 0 0.073 0 -0 0</pose>
         <geometry>
@@ -193,5 +193,5 @@
         </geometry>
       </visual>
-      <visual name='chassis_visual_leg_f_l'>
+      <visual name="chassis_visual_leg_f_l">
         <pose>0.177943 0.19 -0.0987583 0 -0.5 0</pose>
         <geometry>
@@ -202,5 +202,5 @@
         </geometry>
       </visual>
-      <visual name='chassis_visual_leg_f_r'>
+      <visual name="chassis_visual_leg_f_r">
         <pose>0.177943 -0.19 -0.0987583 0 -0.5 0</pose>
         <geometry>
@@ -211,5 +211,5 @@
         </geometry>
       </visual>
-      <visual name='chassis_visual_leg_p_l'>
+      <visual name="chassis_visual_leg_p_l">
         <pose>-0.177943 0.19 -0.0987583 0 0.5 0</pose>
         <geometry>
@@ -220,5 +220,5 @@
         </geometry>
       </visual>
-      <visual name='chassis_visual_leg_p_r'>
+      <visual name="chassis_visual_leg_p_r">
         <pose>-0.177943 -0.19 -0.0987583 0 0.5 0</pose>
         <geometry>
@@ -237,5 +237,5 @@
       <gravity>1</gravity>
     </link>
-    <link name='testa'>
+    <link name="testa">
       <pose>0.2175 -0.012 0.096 0 -0 3.14</pose>
       <inertial>
@@ -251,5 +251,5 @@
         </inertia>
       </inertial>
-      <visual name='testa_visual'>
+      <visual name="testa_visual">
         <pose>0.023 0 0.033 0 -0 0</pose>
         <geometry>
@@ -267,5 +267,5 @@
       <gravity>1</gravity>
     </link>
-    <joint name='pan' type='revolute'>
+    <joint name="pan" type="revolute">
       <child>testa</child>
       <parent>chassis</parent>
@@ -276,9 +276,9 @@
           <upper>1e-16</upper>
         </limit>
-        <dynamics />
+        <dynamics/>
         <use_parent_model_frame>1</use_parent_model_frame>
       </axis>
     </joint>
-    <link name='braccio'>
+    <link name="braccio">
       <pose>0.2175 -0.012 0.14 3.14 -0 3.14</pose>
       <inertial>
@@ -294,5 +294,5 @@
         </inertia>
       </inertial>
-      <collision name='braccio_collision'>
+      <collision name="braccio_collision">
         <pose>0 0 -0.014 0 -0 0</pose>
         <geometry>
@@ -304,13 +304,13 @@
         <surface>
           <contact>
-            <ode />
-          </contact>
-          <bounce />
-          <friction>
-            <ode />
-          </friction>
-        </surface>
-      </collision>
-      <visual name='braccio_visual'>
+            <ode/>
+          </contact>
+          <bounce/>
+          <friction>
+            <ode/>
+          </friction>
+        </surface>
+      </collision>
+      <visual name="braccio_visual">
         <pose>0 0 -0.014 0 -0 0</pose>
         <geometry>
@@ -320,5 +320,5 @@
         </geometry>
       </visual>
-      <visual name='braccio_visual_camera'>
+      <visual name="braccio_visual_camera">
         <pose>1.59519e-05 3.18404e-05 -0.06 1.57159 0.00159265 -1.57159</pose>
         <geometry>
@@ -342,5 +342,5 @@
           </clip>
         </camera>
-        <plugin name="depth_camera_plugin" filename="libgazebo_ros_depth_camera.so">
+        <plugin filename="libgazebo_ros_depth_camera.so" name="depth_camera_plugin">
           <alwaysOn>1</alwaysOn>
           <updateRate>10.0</updateRate>
@@ -390,5 +390,5 @@
           </clip>
         </camera>
-        <plugin name="stereo_camera_controller" filename="libgazebo_ros_multicamera.so">
+        <plugin filename="libgazebo_ros_multicamera.so" name="stereo_camera_controller">
           <alwaysOn>true</alwaysOn>
           <updateRate>0.0</updateRate>
@@ -414,5 +414,5 @@
       <gravity>1</gravity>
     </link>
-    <joint name='tilt' type='revolute'>
+    <joint name="tilt" type="revolute">
       <child>braccio</child>
       <parent>testa</parent>
@@ -423,9 +423,9 @@
           <upper>1e-16</upper>
         </limit>
-        <dynamics />
+        <dynamics/>
         <use_parent_model_frame>1</use_parent_model_frame>
       </axis>
     </joint>
-    <link name='wheel_f_l'>
+    <link name="wheel_f_l">
       <pose>0.225885 0.217 -0.186517 0 -0.5 0</pose>
       <inertial>
@@ -441,5 +441,5 @@
         </inertia>
       </inertial>
-      <collision name='wheel_f_l_collision'>
+      <collision name="wheel_f_l_collision">
         <pose>0 0.035 0 1.57 -0 0</pose>
         <geometry>
@@ -452,13 +452,13 @@
         <surface>
           <contact>
-            <ode />
-          </contact>
-          <bounce />
-          <friction>
-            <ode />
-          </friction>
-        </surface>
-      </collision>
-      <visual name='wheel_f_l_visual'>
+            <ode/>
+          </contact>
+          <bounce/>
+          <friction>
+            <ode/>
+          </friction>
+        </surface>
+      </collision>
+      <visual name="wheel_f_l_visual">
         <pose>0 0.035 0 1.57 -0 0</pose>
         <geometry>
@@ -477,5 +477,5 @@
       <gravity>1</gravity>
     </link>
-    <joint name='shaft_f_l' type='revolute'>
+    <joint name="shaft_f_l" type="revolute">
       <child>wheel_f_l</child>
       <parent>chassis</parent>
@@ -486,9 +486,9 @@
           <upper>1e+16</upper>
         </limit>
-        <dynamics />
+        <dynamics/>
         <use_parent_model_frame>1</use_parent_model_frame>
       </axis>
     </joint>
-    <link name='wheel_f_r'>
+    <link name="wheel_f_r">
       <pose>0.225885 -0.217 -0.186517 0 -0.5 0</pose>
       <inertial>
@@ -504,5 +504,5 @@
         </inertia>
       </inertial>
-      <collision name='wheel_f_r_collision'>
+      <collision name="wheel_f_r_collision">
         <pose>0 -0.035 0 1.57 -0 0</pose>
         <geometry>
@@ -515,13 +515,13 @@
         <surface>
           <contact>
-            <ode />
-          </contact>
-          <bounce />
-          <friction>
-            <ode />
-          </friction>
-        </surface>
-      </collision>
-      <visual name='wheel_f_r_visual'>
+            <ode/>
+          </contact>
+          <bounce/>
+          <friction>
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