Commit message: add rover_amalia_chassis

File: definitions/rover_amalia/model.xacro (robot description, xacro)
@@ -2,20 +2,5 @@
 <sdf version="1.5">
   <model name="rover_amalia">
-    <plugin filename="libgazebo_ros_skid_steer_drive.so" name="skid_steer_drive">
-      <robotNamespace>rover_amalia</robotNamespace>
-      <broadcastTF>1</broadcastTF>
-      <leftFrontJoint>shaft_f_l</leftFrontJoint>
-      <rightFrontJoint>shaft_f_r</rightFrontJoint>
-      <leftRearJoint>shaft_p_l</leftRearJoint>
-      <rightRearJoint>shaft_p_r</rightRearJoint>
-      <wheelSeparation>0.400</wheelSeparation>
-      <wheelDiameter>0.18</wheelDiameter>
-      <torque>5.0</torque>
-      <commandTopic>cmd_vel</commandTopic>
-      <odometryTopic>odom</odometryTopic>
-      <odometryFrame>odom</odometryFrame>
-      <robotBaseFrame>base_footprint</robotBaseFrame>
-      <updateRate>100.0</updateRate>
-    </plugin>
+    <pose>0 0 0 0 0 0</pose>
     <static>0</static>
     <link name="chassis">
@@ -57,80 +42,4 @@
             <size>0.089 0.064 0.046</size>
           </box>
-        </geometry>
-        <max_contacts>10</max_contacts>
-        <surface>
-          <contact>
-            <ode/>
-          </contact>
-          <bounce/>
-          <friction>
-            <ode/>
-          </friction>
-        </surface>
-      </collision>
-      <collision name="chassis_collision_leg_f_l">
-        <pose>0.177943 0.19 -0.0987583 0 -0.5 0</pose>
-        <geometry>
-          <cylinder>
-            <length>0.2</length>
-            <radius>0.008</radius>
-          </cylinder>
-        </geometry>
-        <max_contacts>10</max_contacts>
-        <surface>
-          <contact>
-            <ode/>
-          </contact>
-          <bounce/>
-          <friction>
-            <ode/>
-          </friction>
-        </surface>
-      </collision>
-      <collision name="chassis_collision_leg_f_r">
-        <pose>0.177943 -0.19 -0.0987583 0 -0.5 0</pose>
-        <geometry>
-          <cylinder>
-            <length>0.2</length>
-            <radius>0.008</radius>
-          </cylinder>
-        </geometry>
-        <max_contacts>10</max_contacts>
-        <surface>
-          <contact>
-            <ode/>
-          </contact>
-          <bounce/>
-          <friction>
-            <ode/>
-          </friction>
-        </surface>
-      </collision>
-      <collision name="chassis_collision_leg_p_l">
-        <pose>-0.177943 0.19 -0.0987583 0 0.5 0</pose>
-        <geometry>
-          <cylinder>
-            <length>0.2</length>
-            <radius>0.008</radius>
-          </cylinder>
-        </geometry>
-        <max_contacts>10</max_contacts>
-        <surface>
-          <contact>
-            <ode/>
-          </contact>
-          <bounce/>
-          <friction>
-            <ode/>
-          </friction>
-        </surface>
-      </collision>
-      <collision name="chassis_collision_leg_p_r">
-        <pose>-0.177943 -0.19 -0.0987583 0 0.5 0</pose>
-        <geometry>
-          <cylinder>
-            <length>0.2</length>
-            <radius>0.008</radius>
-          </cylinder>
         </geometry>
         <max_contacts>10</max_contacts>
@@ -193,491 +102,24 @@
         </geometry>
       </visual>
-      <visual name="chassis_visual_leg_f_l">
-        <pose>0.177943 0.19 -0.0987583 0 -0.5 0</pose>
-        <geometry>
-          <cylinder>
-            <length>0.2</length>
-            <radius>0.008</radius>
-          </cylinder>
-        </geometry>
-      </visual>
-      <visual name="chassis_visual_leg_f_r">
-        <pose>0.177943 -0.19 -0.0987583 0 -0.5 0</pose>
-        <geometry>
-          <cylinder>
-            <length>0.2</length>
-            <radius>0.008</radius>
-          </cylinder>
-        </geometry>
-      </visual>
-      <visual name="chassis_visual_leg_p_l">
-        <pose>-0.177943 0.19 -0.0987583 0 0.5 0</pose>
-        <geometry>
-          <cylinder>
-            <length>0.2</length>
-            <radius>0.008</radius>
-          </cylinder>
-        </geometry>
-      </visual>
-      <visual name="chassis_visual_leg_p_r">
-        <pose>-0.177943 -0.19 -0.0987583 0 0.5 0</pose>
-        <geometry>
-          <cylinder>
-            <length>0.2</length>
-            <radius>0.008</radius>
-          </cylinder>
-        </geometry>
-      </visual>
-      <velocity_decay>
-        <linear>0</linear>
-        <angular>0</angular>
-      </velocity_decay>
       <self_collide>0</self_collide>
       <kinematic>0</kinematic>
       <gravity>1</gravity>
     </link>
-    <link name="testa">
-      <pose>0.2175 -0.012 0.096 0 -0 3.14</pose>
-      <inertial>
-        <pose>0 0 0 0 -0 0</pose>
-        <mass>1</mass>
-        <inertia>
-          <ixx>100</ixx>
-          <ixy>0</ixy>
-          <ixz>0</ixz>
-          <iyy>100</iyy>
-          <iyz>0</iyz>
-          <izz>100</izz>
-        </inertia>
-      </inertial>
-      <visual name="testa_visual">
-        <pose>0.023 0 0.033 0 -0 0</pose>
-        <geometry>
-          <box>
-            <size>0.09 0.043 0.066</size>
-          </box>
-        </geometry>
-      </visual>
-      <velocity_decay>
-        <linear>0</linear>
-        <angular>0</angular>
-      </velocity_decay>
-      <self_collide>0</self_collide>
-      <kinematic>0</kinematic>
-      <gravity>1</gravity>
-    </link>
-    <joint name="pan" type="revolute">
-      <child>testa</child>
-      <parent>chassis</parent>
-      <axis>
-        <xyz>0 0 1</xyz>
-        <limit>
-          <lower>-1e-16</lower>
-          <upper>1e-16</upper>
-        </limit>
-        <dynamics/>
-        <use_parent_model_frame>1</use_parent_model_frame>
-      </axis>
-    </joint>
-    <link name="braccio">
-      <pose>0.2175 -0.012 0.14 3.14 -0 3.14</pose>
-      <inertial>
-        <pose>0 0 -0.02 0 -0 0</pose>
-        <mass>2</mass>
-        <inertia>
-          <ixx>200.001</ixx>
-          <ixy>0</ixy>
-          <ixz>0</ixz>
-          <iyy>200.001</iyy>
-          <iyz>0</iyz>
-          <izz>200</izz>
-        </inertia>
-      </inertial>
-      <collision name="braccio_collision">
-        <pose>0 0 -0.014 0 -0 0</pose>
-        <geometry>
-          <box>
-            <size>0.02 0.061 0.049</size>
-          </box>
-        </geometry>
-        <max_contacts>10</max_contacts>
-        <surface>
-          <contact>
-            <ode/>
-          </contact>
-          <bounce/>
-          <friction>
-            <ode/>
-          </friction>
-        </surface>
-      </collision>
-      <visual name="braccio_visual">
-        <pose>0 0 -0.014 0 -0 0</pose>
-        <geometry>
-          <box>
-            <size>0.02 0.061 0.049</size>
-          </box>
-        </geometry>
-      </visual>
-      <visual name="braccio_visual_camera">
-        <pose>1.59519e-05 3.18404e-05 -0.06 1.57159 0.00159265 -1.57159</pose>
-        <geometry>
-          <box>
-            <size>0.2 0.04 0.04</size>
-          </box>
-        </geometry>
-      </visual>
-      <sensor name="depth_camera" type="depth">
-        <pose>0.0 0.0 0.0 0.0 3.14 0.0</pose>
-        <camera>
-          <horizontal_fov>1.578</horizontal_fov>
-          <image>
-            <width>640</width>
-            <height>480</height>
-            <format>R8G8B8</format>
-          </image>
-          <clip>
-            <near>0.4</near>
-            <far>100</far>
-          </clip>
-        </camera>
-        <plugin filename="libgazebo_ros_depth_camera.so" name="depth_camera_plugin">
-          <alwaysOn>1</alwaysOn>
-          <updateRate>10.0</updateRate>
-          <imageTopicName>image_raw</imageTopicName>
-          <depthImageTopicName>depth_raw</depthImageTopicName>
-          <depthImageCameraInfoTopicName>camera_info</depthImageCameraInfoTopicName>
-          <pointCloudTopicName>points</pointCloudTopicName>
-          <cameraInfoTopicName>camera_info</cameraInfoTopicName>
-          <cameraName>depth_cam</cameraName>
-          <frameName>/base_link</frameName>
-          <pointCloudCutoff>0.001</pointCloudCutoff>
-          <distortionK1>0.0</distortionK1>
-          <distortionK2>0.0</distortionK2>
-          <distortionK3>0.0</distortionK3>
-          <distortionT1>0.0</distortionT1>
-          <distortionT2>0.0</distortionT2>
-        </plugin>
-        <always_on>true</always_on>
-        <update_rate>10.0</update_rate>
-      </sensor>
-      <sensor name="camera" type="multicamera">
-        <always_on>1</always_on>
-        <update_rate>30</update_rate>
-        <visualize>true</visualize>
-        <camera name="left">
-          <pose>0 0 0 0 3.14 0</pose>
-          <horizontal_fov>1.047</horizontal_fov>
-          <image>
-            <width>320</width>
-            <height>240</height>
-          </image>
-          <clip>
-            <near>0.4</near>
-            <far>100</far>
-          </clip>
-        </camera>
-        <camera name="right">
-          <pose>0 -0.2 0 0 3.14 0</pose>
-          <horizontal_fov>1.047</horizontal_fov>
-          <image>
-            <width>320</width>
-            <height>240</height>
-          </image>
-          <clip>
-            <near>0.4</near>
-            <far>100</far>
-          </clip>
-        </camera>
-        <plugin filename="libgazebo_ros_multicamera.so" name="stereo_camera_controller">
-          <alwaysOn>true</alwaysOn>
-          <updateRate>0.0</updateRate>
-          <cameraName>camera</cameraName>
-          <imageTopicName>image_raw</imageTopicName>
-          <cameraInfoTopicName>camera_info</cameraInfoTopicName>
-          <frameName>left_camera_optical_frame</frameName>
-          <!--<rightFrameName>right_camera_optical_frame</rightFrameName>-->
-          <hackBaseline>0.07</hackBaseline>
-          <distortionK1>0.0</distortionK1>
-          <distortionK2>0.0</distortionK2>
-          <distortionK3>0.0</distortionK3>
-          <distortionT1>0.0</distortionT1>
-          <distortionT2>0.0</distortionT2>
-        </plugin>
-      </sensor>
-      <velocity_decay>
-        <linear>0</linear>
-        <angular>0</angular>
-      </velocity_decay>
-      <self_collide>0</self_collide>
-      <kinematic>0</kinematic>
-      <gravity>1</gravity>
-    </link>
-    <joint name="tilt" type="revolute">
-      <child>braccio</child>
-      <parent>testa</parent>
-      <axis>
-        <xyz>-0.001593 -0.999997 -0.001593</xyz>
-        <limit>
-          <lower>-1e-16</lower>
-          <upper>1e-16</upper>
-        </limit>
-        <dynamics/>
-        <use_parent_model_frame>1</use_parent_model_frame>
-      </axis>
-    </joint>
-    <link name="wheel_f_l">
-      <pose>0.225885 0.217 -0.186517 0 -0.5 0</pose>
-      <inertial>
-        <pose>0 0 0 0 -0 0</pose>
-        <mass>1</mass>
-        <inertia>
-          <ixx>100</ixx>
-          <ixy>0</ixy>
-          <ixz>0</ixz>
-          <iyy>100</iyy>
-          <iyz>0</iyz>
-          <izz>100</izz>
-        </inertia>
-      </inertial>
-      <collision name="wheel_f_l_collision">
-        <pose>0 0.035 0 1.57 -0 0</pose>
-        <geometry>
-          <cylinder>
-            <length>0.07</length>
-            <radius>0.09</radius>
-          </cylinder>
-        </geometry>
-        <max_contacts>10</max_contacts>
-        <surface>
-          <contact>
-            <ode/>
-          </contact>
-          <bounce/>
-          <friction>
-            <ode/>
-          </friction>
-        </surface>
-      </collision>
-      <visual name="wheel_f_l_visual">
-        <pose>0 0.035 0 1.57 -0 0</pose>
-        <geometry>
-          <cylinder>
-            <length>0.07</length>
-            <radius>0.09</radius>
-          </cylinder>
-        </geometry>
-      </visual>
-      <velocity_decay>
-        <linear>0</linear>
-        <angular>0</angular>
-      </velocity_decay>
-      <self_collide>0</self_collide>
-      <kinematic>0</kinematic>
-      <gravity>1</gravity>
-    </link>
-    <joint name="shaft_f_l" type="revolute">
-      <child>wheel_f_l</child>
-      <parent>chassis</parent>
-      <axis>
-        <xyz>0 1 0</xyz>
-        <limit>
-          <lower>-1e+16</lower>
-          <upper>1e+16</upper>
-        </limit>
-        <dynamics/>
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
File: definitions/rover_amalia_leg/model.xacro (robot description, xacro)
@@ -2,6 +2,6 @@
 <sdf version="1.5" xmlns:xacro="http://www.ros.org/wiki/xacro">
   <xacro:include filename="./rover_amalia_leg.xacro" />
-  <model name="rover_amalia">
-    <xacro:leg prefix="f_r" reflect_xz="1" reflect_yz="1" bar_length="0.2" bar_radius="0.008" wheel_radius="0.08" wheel_length="0.07"/>
+  <model name="rover_amalia_leg">
+    <xacro:rover_amalia_leg prefix="f_r" reflect_xz="1" reflect_yz="1" bar_length="0.2" bar_radius="0.008" wheel_radius="0.08" wheel_length="0.07"/>
     <pose>0 0 0 0 0 0</pose>
   </model>

File: definitions/rover_amalia_leg/rover_amalia_leg.xacro (robot description, xacro)
@@ -1,5 +1,5 @@
 <?xml version="1.0" ?>
 <robot name="rover_amalia_leg" xmlns:xacro="http://www.ros.org/wiki/xacro">
-  <xacro:macro name="leg" params="prefix reflect_xz reflect_yz bar_length bar_radius wheel_radius wheel_length">
+  <xacro:macro name="rover_amalia_leg" params="prefix reflect_xz reflect_yz bar_length bar_radius wheel_radius wheel_length">
     <link name="leg_bar_${prefix}">
     <collision name="leg_bar_${prefix}_bar_collision">
@@ -33,5 +33,5 @@
   </link>
   <link name="leg_wheel_${prefix}">
-    <pose>${0.225885*reflect_yz} ${(-0.217)*reflect_xz} -0.186517 0 ${(-0.5)*reflect_yz} 0</pose>
+    <pose>${0.225885*reflect_yz} ${(-0.205)*reflect_xz} -0.186517 0 ${(-0.5)*reflect_yz} 0</pose>
     <inertial>
       <pose>0 0 0 0 -0 0</pose>

File: definitions/rover_amalia_turret/model.xacro (robot description, xacro)
@@ -2,6 +2,6 @@
 <sdf version="1.5" xmlns:xacro="http://www.ros.org/wiki/xacro">
   <xacro:include filename="./rover_amalia_turret.xacro" />
-  <model name="rover_amalia">
-    <xacro:turret Ox="1" Oy="1" Oz="1" bar_height="0.2"/>
+  <model name="rover_amalia_turret">
+    <xacro:rover_amalia_turret Ox="0" Oy="0" Oz="0" bar_height="0.2"/>
     <pose>0 0 0 0 0 0</pose>
   </model>

File: definitions/rover_amalia_turret/rover_amalia_turret.xacro (robot description, xacro)
@@ -20,5 +20,5 @@
     <size>0.06 0.02 ${rover_amalia_turret_pan_tilt_height}</size>
   </xacro:property>
-  <xacro:macro name="turret" params="Ox Oy Oz bar_height">
+  <xacro:macro name="rover_amalia_turret" params="Ox Oy Oz bar_height">
     <link name="rover_amalia_turret_bar">
       <xacro:insert_block name="rover_amalia_turret_bar_pose"/>
