Commit message: fix rover_amalia

File: definitions/rover_amalia/model.xacro (robot description, xacro)
@@ -1,118 +1,71 @@
 <?xml version="1.0" ?>
-<sdf version="1.5">
+<sdf version="1.5" xmlns:xacro="http://www.ros.org/wiki/xacro">
+  <xacro:include filename="../rover_amalia_leg/rover_amalia_leg.xacro"/>
+  <xacro:include filename="../rover_amalia_chassis/rover_amalia_chassis.xacro"/>
+  <xacro:include filename="../rover_amalia_turret/rover_amalia_turret.xacro"/>
+  <xacro:property name="leg_bar_length" value="0.2"/>
+  <xacro:property name="leg_bar_radius" value="0.008"/>
+  <xacro:property name="wheel_radius" value="0.08"/>
+  <xacro:property name="wheel_length" value="0.07"/>
+  <xacro:property name="turret_base_x" value="0.195"/>
+  <xacro:property name="chassis_size_x" value="0.492"/>
+  <xacro:property name="chassis_size_y" value="0.334"/>
+  <xacro:property name="chassis_size_z" value="0.1"/>
+  <xacro:property name="chassis_height" value="${leg_bar_length+wheel_radius}"/>
+  <xacro:property name="leg_x" value="${chassis_size_x*3/8}"/>
+  <xacro:property name="leg_y" value="${chassis_size_y/2 + leg_bar_radius}"/>
+  <xacro:macro name="rover_amalia_joint_chassis_leg" params="prefix reflect_xz reflect_yz">
+    <joint name="rover_amalia_joint_chassis_leg_${prefix}" type="revolute">
+      <child>rover_amalia_leg_bar_${prefix}</child>
+      <parent>rover_amalia_chassis</parent>
+      <axis>
+        <xyz>0 1 0</xyz>
+        <limit>
+          <lower>-1e-16</lower>
+          <upper>1e-16</upper>
+        </limit>
+        <dynamics/>
+        <use_parent_model_frame>1</use_parent_model_frame>
+      </axis>
+    </joint>
+  </xacro:macro>
   <model name="rover_amalia">
     <pose>0 0 0 0 0 0</pose>
     <static>0</static>
-    <link name="chassis">
-      <pose>0 0 0 0 0 0</pose>
-      <inertial>
-        <pose>0.0216667 0 -0.0215556 0 -0 0</pose>
-        <mass>9</mass>
-        <inertia>
-          <ixx>900.12</ixx>
-          <ixy>-3.46945e-18</ixy>
-          <ixz>-0.0139533</ixz>
-          <iyy>900.352</iyy>
-          <iyz>0</iyz>
-          <izz>900.455</izz>
-        </inertia>
-      </inertial>
-      <collision name="chassis_collision">
-        <pose>0 0 0 0 -0 0</pose>
-        <geometry>
-          <box>
-            <size>0.492 0.334 0.1</size>
-          </box>
-        </geometry>
-        <max_contacts>10</max_contacts>
-        <surface>
-          <contact>
-            <ode/>
-          </contact>
-          <bounce/>
-          <friction>
-            <ode/>
-          </friction>
-        </surface>
-      </collision>
-      <collision name="chassis_collision_base">
-        <pose>0.195 0 0.073 0 -0 0</pose>
-        <geometry>
-          <box>
-            <size>0.089 0.064 0.046</size>
-          </box>
-        </geometry>
-        <max_contacts>10</max_contacts>
-        <surface>
-          <contact>
-            <ode/>
-          </contact>
-          <bounce/>
-          <friction>
-            <ode/>
-          </friction>
-        </surface>
-      </collision>
-      <visual name="chassis_visual">
-        <pose>0 0 0 0 -0 0</pose>
-        <geometry>
-          <box>
-            <size>0.492 0.334 0.1</size>
-          </box>
-        </geometry>
-      </visual>
-      <visual name="chassis_visual_Range_Front">
-        <pose>0.246 0 -0.05 0 -0 0</pose>
-        <geometry>
-          <box>
-            <size>0.01 0.03 0.01</size>
-          </box>
-        </geometry>
-      </visual>
-      <visual name="chassis_visual_Range_Front_Down">
-        <pose>0.246 0 -0.05 0 1.57 0</pose>
-        <geometry>
-          <box>
-            <size>0.01 0.03 0.01</size>
-          </box>
-        </geometry>
-      </visual>
-      <visual name="chassis_visual_Range_Post">
-        <pose>-0.246 0 -0.05 3.14159 0.00159265 3.14159</pose>
-        <geometry>
-          <box>
-            <size>0.01 0.03 0.01</size>
-          </box>
-        </geometry>
-      </visual>
-      <visual name="chassis_visual_Range_Post_Down">
-        <pose>-0.246 0 -0.05 0 1.57 0</pose>
-        <geometry>
-          <box>
-            <size>0.01 0.03 0.01</size>
-          </box>
-        </geometry>
-      </visual>
-      <visual name="chassis_visual_base">
-        <pose>0.195 0 0.073 0 -0 0</pose>
-        <geometry>
-          <box>
-            <size>0.089 0.064 0.046</size>
-          </box>
-        </geometry>
-      </visual>
-      <self_collide>0</self_collide>
-      <kinematic>0</kinematic>
-      <gravity>1</gravity>
-    </link>
+    <!--main components-->
+    <xacro:rover_amalia_turret Ox="${turret_base_x}" Oy="0" Oz="${chassis_height+0.1}" bar_height="0.2"/>
+    <xacro:rover_amalia_chassis Ox="0" Oy="0" Oz="${chassis_height}" body_size_x="${chassis_size_x}" body_size_y="${chassis_size_y}" body_size_z="${chassis_size_z}" turret_base_x="${turret_base_x}" turret_base_y="0"/>
+    <xacro:rover_amalia_leg Ox="${leg_x}" Oy="${leg_y}" Oz="0" prefix="f_r" reflect_xz="1" reflect_yz="1" bar_length="${leg_bar_length}" bar_radius="${leg_bar_radius}" wheel_radius="${wheel_radius}" wheel_length="${wheel_length}"/>
+    <xacro:rover_amalia_leg Ox="${leg_x}" Oy="${leg_y}" Oz="0" prefix="f_l" reflect_xz="-1" reflect_yz="1" bar_length="${leg_bar_length}" bar_radius="${leg_bar_radius}" wheel_radius="${wheel_radius}" wheel_length="${wheel_length}"/>
+    <xacro:rover_amalia_leg Ox="${leg_x}" Oy="${leg_y}" Oz="0" prefix="b_r" reflect_xz="1" reflect_yz="-1" bar_length="${leg_bar_length}" bar_radius="${leg_bar_radius}" wheel_radius="${wheel_radius}" wheel_length="${wheel_length}"/>
+    <xacro:rover_amalia_leg Ox="${leg_x}" Oy="${leg_y}" Oz="0" prefix="b_l" reflect_xz="-1" reflect_yz="-1" bar_length="${leg_bar_length}" bar_radius="${leg_bar_radius}" wheel_radius="${wheel_radius}" wheel_length="${wheel_length}"/>
+    <!--additional joints-->
+    <xacro:rover_amalia_joint_chassis_leg prefix="f_r" reflect_xz="1" reflect_yz="1"/>
+    <xacro:rover_amalia_joint_chassis_leg prefix="f_l" reflect_xz="-1" reflect_yz="1"/>
+    <xacro:rover_amalia_joint_chassis_leg prefix="b_r" reflect_xz="1" reflect_yz="-1"/>
+    <xacro:rover_amalia_joint_chassis_leg prefix="b_l" reflect_xz="-1" reflect_yz="-1"/>
+    <joint name="rover_amalia_joint_turret_base_turret" type="revolute">
+      <child>rover_amalia_turret_bar</child>
+      <parent>rover_amalia_chassis</parent>
+      <axis>
+        <xyz>0 0 1</xyz>
+        <limit>
+          <lower>-1e-16</lower>
+          <upper>1e-16</upper>
+        </limit>
+        <dynamics/>
+        <use_parent_model_frame>1</use_parent_model_frame>
+      </axis>
+    </joint>
+    <!--additional plugins-->
     <plugin filename="libgazebo_ros_skid_steer_drive.so" name="skid_steer_drive">
       <robotNamespace>rover_amalia</robotNamespace>
       <broadcastTF>1</broadcastTF>
-      <leftFrontJoint>shaft_f_l</leftFrontJoint>
-      <rightFrontJoint>shaft_f_r</rightFrontJoint>
-      <leftRearJoint>shaft_p_l</leftRearJoint>
-      <rightRearJoint>shaft_p_r</rightRearJoint>
+      <rightFrontJoint>rover_amalia_leg_shaft_f_r</rightFrontJoint>
+      <leftFrontJoint>rover_amalia_leg_shaft_f_l</leftFrontJoint>
+      <rightRearJoint>rover_amalia_leg_shaft_b_r</rightRearJoint>
+      <leftRearJoint>rover_amalia_leg_shaft_b_l</leftRearJoint>
       <wheelSeparation>0.400</wheelSeparation>
-      <wheelDiameter>0.18</wheelDiameter>
+      <wheelDiameter>${wheel_radius*2}</wheelDiameter>
       <torque>5.0</torque>
       <commandTopic>cmd_vel</commandTopic>

File: definitions/rover_amalia_chassis/model.xacro (robot description, xacro)
@@ -3,5 +3,5 @@
   <xacro:include filename="./rover_amalia_chassis.xacro" />
   <model name="rover_amalia_chassis">
-    <xacro:rover_amalia_chassis Ox="0" Oy="0" Oz="0"/>
+    <xacro:rover_amalia_chassis Ox="0" Oy="0" Oz="0" body_size_x="0.492" body_size_y="0.334" body_size_z="0.1" turret_base_x="0.195" turret_base_y="0"/>
     <pose>0 0 0 0 0 0</pose>
   </model>

File: definitions/rover_amalia_chassis/rover_amalia_chassis.xacro (robot description, xacro)
@@ -2,12 +2,10 @@
 <robot name="rover_amalia_chassis" xmlns:xacro="http://www.ros.org/wiki/xacro">
   <xacro:property name="pi" value="3.1415926"/>
-  <xacro:property name="rover_amalia_chassis_turret_base_pose">
-     <pose>0.195 0 0.073 0 -0 0</pose>
-  </xacro:property>
   <xacro:property name="rover_amalia_chassis_turret_base_size">
      <size>0.089 0.064 0.046</size>
   </xacro:property>
   <xacro:property name="rover_amalia_chassis_body_size">
-     <size>0.492 0.334 0.1</size>
+     <!--<size>0.492 0.334 0.1</size>-->
+     <size>${body_size_x} ${body_size_y} ${body_size_z}</size>
   </xacro:property>
   <xacro:property name="rover_amalia_chassis_rangefinder_size_y" value="0.01"/>
@@ -15,7 +13,8 @@
     <size>${rover_amalia_chassis_rangefinder_size_y} 0.03 ${rover_amalia_chassis_rangefinder_size_y}</size>
   </xacro:property>
-  <xacro:macro name="rover_amalia_chassis" params="Ox Oy Oz">
+  <xacro:property name="rover_amalia_chassis_turret_base_z" value="0.073"/>
+  <xacro:macro name="rover_amalia_chassis" params="Ox Oy Oz body_size_x body_size_y body_size_z turret_base_x turret_base_y">
     <link name="rover_amalia_chassis">
-      <pose>0 0 0 0 0 0</pose>
+      <pose>${Ox} ${Oy} ${Oz} 0 0 0</pose>
       <inertial>
         <pose>0.0216667 0 -0.0215556 0 -0 0</pose>
@@ -30,9 +29,17 @@
         </inertia>
       </inertial>
-      <collision name="rover_amalia_chassis_collision">
+      <visual name="rover_amalia_chassis_body_visual">
         <pose>0 0 0 0 0 0</pose>
         <geometry>
           <box>
-            <size>0.492 0.334 0.1</size>
+            <xacro:insert_block name="rover_amalia_chassis_body_size"/>
+          </box>
+        </geometry>
+      </visual>
+      <collision name="rover_amalia_chassis_body_collision">
+        <pose>0 0 0 0 0 0</pose>
+        <geometry>
+          <box>
+            <xacro:insert_block name="rover_amalia_chassis_body_size"/>
           </box>
         </geometry>
@@ -40,5 +47,5 @@
       </collision>
       <collision name="rover_amalia_chassis_turret_base_collision">
-        <xacro:insert_block name="rover_amalia_chassis_turret_base_pose"/>
+        <pose>${turret_base_x} ${turret_base_y} ${rover_amalia_chassis_turret_base_z} 0 0 0</pose>
         <geometry>
           <box>
@@ -49,16 +56,8 @@
       </collision>
       <visual name="rover_amalia_chassis_turret_base_visual">
-        <xacro:insert_block name="rover_amalia_chassis_turret_base_pose"/>
+        <pose>${turret_base_x} ${turret_base_y} ${rover_amalia_chassis_turret_base_z} 0 0 0</pose>
         <geometry>
           <box>
             <xacro:insert_block name="rover_amalia_chassis_turret_base_size"/>
-          </box>
-        </geometry>
-      </visual>
-      <visual name="rover_amalia_chassis_body_visual">
-        <pose>0 0 0 0 0 0</pose>
-        <geometry>
-          <box>
-            <xacro:insert_block name="rover_amalia_chassis_body_size"/>
           </box>
         </geometry>

File: definitions/rover_amalia_leg/model.xacro (robot description, xacro)
@@ -3,6 +3,6 @@
   <xacro:include filename="./rover_amalia_leg.xacro" />
   <model name="rover_amalia_leg">
-    <xacro:rover_amalia_leg prefix="f_r" reflect_xz="1" reflect_yz="1" bar_length="0.2" bar_radius="0.008" wheel_radius="0.08" wheel_length="0.07"/>
     <pose>0 0 0 0 0 0</pose>
+    <xacro:rover_amalia_leg Ox="0" Oy="0" Oz="0" prefix="f_r" reflect_xz="1" reflect_yz="1" bar_length="0.2" bar_radius="0.008" wheel_radius="0.08" wheel_length="0.07"/>
   </model>
 </sdf>

File: definitions/rover_amalia_leg/rover_amalia_leg.xacro (robot description, xacro)
@@ -1,8 +1,10 @@
 <?xml version="1.0" ?>
 <robot name="rover_amalia_leg" xmlns:xacro="http://www.ros.org/wiki/xacro">
-  <xacro:macro name="rover_amalia_leg" params="prefix reflect_xz reflect_yz bar_length bar_radius wheel_radius wheel_length">
-    <link name="leg_bar_${prefix}">
+  <xacro:property name="pi" value="3.1415926" />
+  <xacro:property name="rover_amalia_leg_bar_z" value="${wheel_radius+bar_length/2}" />
+  <xacro:macro name="rover_amalia_leg" params="Ox Oy Oz prefix reflect_xz reflect_yz bar_length bar_radius wheel_radius wheel_length">
+    <link name="rover_amalia_leg_bar_${prefix}">
+      <pose>${Ox*reflect_yz} ${Oy*reflect_xz} ${Oz+rover_amalia_leg_bar_z} 0 0 0</pose>
     <collision name="leg_bar_${prefix}_bar_collision">
-      <pose>${0.177943*reflect_yz} ${(-0.19)*reflect_xz} -0.0987583 0 ${(-0.5)*reflect_yz} 0</pose>
       <geometry>
         <cylinder>
@@ -22,6 +24,6 @@
       </surface>
     </collision>
-    <visual name="leg_bar_${prefix}_bar_visual">
-      <pose>${0.177943*reflect_yz} ${(-0.19)*reflect_xz} -0.0987583 0 ${(-0.5)*reflect_yz} 0</pose>
+    <visual name="rover_amalia_leg_bar_${prefix}_bar_visual">
+      <pose>0 0 0 0 0 0</pose>
       <geometry>
         <cylinder>
@@ -32,8 +34,8 @@
     </visual>
   </link>
-  <link name="leg_wheel_${prefix}">
-    <pose>${0.225885*reflect_yz} ${(-0.205)*reflect_xz} -0.186517 0 ${(-0.5)*reflect_yz} 0</pose>
+  <link name="rover_amalia_leg_wheel_${prefix}">
+    <pose>${Ox*reflect_yz} ${(Oy+wheel_length/2+bar_radius+0.001)*reflect_xz} ${wheel_radius} 0 0 0</pose>
     <inertial>
-      <pose>0 0 0 0 -0 0</pose>
+      <pose>0 0 0 0 0 0</pose>
       <mass>1</mass>
       <inertia>
@@ -46,6 +48,6 @@
       </inertia>
     </inertial>
-    <collision name="leg_wheel_${prefix}_collision">
-      <pose>0 ${(-0.035)*reflect_xz} 0 1.57 -0 0</pose>
+    <collision name="rover_amalia_leg_wheel_${prefix}_collision">
+      <pose>0 0 0 ${pi/2} 0 0</pose>
       <geometry>
         <cylinder>
@@ -55,16 +57,7 @@
       </geometry>
       <max_contacts>10</max_contacts>
-      <surface>
-        <contact>
-          <ode/>
-        </contact>
-        <bounce/>
-        <friction>
-          <ode/>
-        </friction>
-      </surface>
     </collision>
-    <visual name="leg_wheel_${prefix}_visual">
-      <pose>0 ${(-0.035)*reflect_xz} 0 1.57 -0 0</pose>
+    <visual name="rover_amalia_leg_wheel_${prefix}_visual">
+      <pose>0 0 0 ${pi/2} 0 0</pose>
       <geometry>
         <cylinder>
@@ -74,15 +67,11 @@
       </geometry>
     </visual>
-    <velocity_decay>
-      <linear>0</linear>
-      <angular>0</angular>
-    </velocity_decay>
     <self_collide>0</self_collide>
     <kinematic>0</kinematic>
     <gravity>1</gravity>
   </link>
-  <joint name="leg_shaft_${prefix}" type="revolute">
-    <child>leg_wheel_${prefix}</child>
-    <parent>leg_bar_${prefix}</parent>
+  <joint name="rover_amalia_leg_shaft_${prefix}" type="revolute">
+    <child>rover_amalia_leg_wheel_${prefix}</child>
+    <parent>rover_amalia_leg_bar_${prefix}</parent>
     <axis>
       <xyz>0 1 0</xyz>
@@ -91,5 +80,4 @@
         <upper>1e+16</upper>
       </limit>
-      <dynamics/>
       <use_parent_model_frame>1</use_parent_model_frame>
     </axis>

Commit message: add chassis size

File: definitions/rover_amalia/model.xacro (robot description, xacro)
@@ -66,7 +66,7 @@
       <rightRearJoint>rover_amalia_leg_shaft_b_r</rightRearJoint>
       <leftRearJoint>rover_amalia_leg_shaft_b_l</leftRearJoint>
-      <wheelSeparation>0.400</wheelSeparation>
+      <wheelSeparation>${chassis_size_x}</wheelSeparation>
       <wheelDiameter>${wheel_radius*2}</wheelDiameter>
-      <torque>5.0</torque>
+      <torque>50.0</torque>
       <commandTopic>cmd_vel</commandTopic>
       <odometryTopic>odom</odometryTopic>

File: definitions/rover_amalia_chassis/rover_amalia_chassis.xacro (robot description, xacro)
@@ -19,5 +19,6 @@
       <inertial>
         <pose>0.0216667 0 -0.0215556 0 -0 0</pose>
-        <mass>9</mass>
+        <!--temporary set the mass to 1000, change when all the inertial will be ok-->
+        <mass>100</mass>
         <inertia>
           <ixx>900.12</ixx>
