Commit message: add meshes

File: definitions/rover_amalia/model.xacro (robot description, xacro)
@@ -4,5 +4,5 @@
   <xacro:include filename="../rover_amalia_chassis/rover_amalia_chassis.xacro"/>
   <xacro:include filename="../rover_amalia_turret/rover_amalia_turret.xacro"/>
-  <xacro:property name="leg_bar_length" value="0.2"/>
+  <xacro:property name="leg_bar_length" value="0.22"/>
   <xacro:property name="leg_bar_radius" value="0.008"/>
   <xacro:property name="wheel_radius" value="0.08"/>
@@ -11,7 +11,7 @@
   <xacro:property name="chassis_size_x" value="0.492"/>
   <xacro:property name="chassis_size_y" value="0.334"/>
-  <xacro:property name="chassis_size_z" value="0.1"/>
-  <xacro:property name="chassis_height" value="${leg_bar_length+wheel_radius}"/>
-  <xacro:property name="leg_x" value="${chassis_size_x*3/8}"/>
+  <xacro:property name="chassis_size_z" value="0.215"/>
+  <xacro:property name="chassis_height" value="${leg_bar_length+wheel_radius+0.05}"/>
+  <xacro:property name="leg_x" value="${chassis_size_x*0.27}"/>
   <xacro:property name="leg_y" value="${chassis_size_y/2 + leg_bar_radius}"/>
   <xacro:macro name="rover_amalia_joint_chassis_leg" params="prefix reflect_xz reflect_yz">
@@ -35,9 +35,9 @@
     <!--main components-->
     <xacro:rover_amalia_turret Ox="${turret_base_x}" Oy="0" Oz="${chassis_height+0.1}" bar_height="0.2"/>
-    <xacro:rover_amalia_chassis Ox="0" Oy="0" Oz="${chassis_height}" body_size_x="${chassis_size_x}" body_size_y="${chassis_size_y}" body_size_z="${chassis_size_z}" turret_base_x="${turret_base_x}" turret_base_y="0"/>
-    <xacro:rover_amalia_leg Ox="${leg_x}" Oy="${leg_y}" Oz="0" prefix="f_r" reflect_xz="1" reflect_yz="1" bar_length="${leg_bar_length}" bar_radius="${leg_bar_radius}" wheel_radius="${wheel_radius}" wheel_length="${wheel_length}"/>
-    <xacro:rover_amalia_leg Ox="${leg_x}" Oy="${leg_y}" Oz="0" prefix="f_l" reflect_xz="-1" reflect_yz="1" bar_length="${leg_bar_length}" bar_radius="${leg_bar_radius}" wheel_radius="${wheel_radius}" wheel_length="${wheel_length}"/>
-    <xacro:rover_amalia_leg Ox="${leg_x}" Oy="${leg_y}" Oz="0" prefix="b_r" reflect_xz="1" reflect_yz="-1" bar_length="${leg_bar_length}" bar_radius="${leg_bar_radius}" wheel_radius="${wheel_radius}" wheel_length="${wheel_length}"/>
-    <xacro:rover_amalia_leg Ox="${leg_x}" Oy="${leg_y}" Oz="0" prefix="b_l" reflect_xz="-1" reflect_yz="-1" bar_length="${leg_bar_length}" bar_radius="${leg_bar_radius}" wheel_radius="${wheel_radius}" wheel_length="${wheel_length}"/>
+    <xacro:rover_amalia_chassis Ox="0" Oy="0" Oz="${chassis_height}" body_size_x="${chassis_size_x}" body_size_y="${chassis_size_y}" body_size_z="${chassis_size_z}" turret_base_x="${turret_base_x}" turret_base_y="0.05"/>
+    <xacro:rover_amalia_leg Ox="${leg_x}" Oy="${leg_y}" Oz="0" prefix="f_r" reflect_xz="1" reflect_yz="1" bar_length="${leg_bar_length}" bar_radius="${leg_bar_radius}" wheel_radius="${wheel_radius}" wheel_length="${wheel_length}" model_root="rover_amalia_leg"/>
+    <xacro:rover_amalia_leg Ox="${leg_x}" Oy="${leg_y}" Oz="0" prefix="f_l" reflect_xz="-1" reflect_yz="1" bar_length="${leg_bar_length}" bar_radius="${leg_bar_radius}" wheel_radius="${wheel_radius}" wheel_length="${wheel_length}" model_root="rover_amalia_leg"/>
+    <xacro:rover_amalia_leg Ox="${leg_x}" Oy="${leg_y}" Oz="0" prefix="b_r" reflect_xz="1" reflect_yz="-1" bar_length="${leg_bar_length}" bar_radius="${leg_bar_radius}" wheel_radius="${wheel_radius}" wheel_length="${wheel_length}" model_root="rover_amalia_leg"/>
+    <xacro:rover_amalia_leg Ox="${leg_x}" Oy="${leg_y}" Oz="0" prefix="b_l" reflect_xz="-1" reflect_yz="-1" bar_length="${leg_bar_length}" bar_radius="${leg_bar_radius}" wheel_radius="${wheel_radius}" wheel_length="${wheel_length}" model_root="rover_amalia_leg"/>
     <!--additional joints-->
     <xacro:rover_amalia_joint_chassis_leg prefix="f_r" reflect_xz="1" reflect_yz="1"/>

File: definitions/rover_amalia_chassis/model.xacro (robot description, xacro)
@@ -3,5 +3,5 @@
   <xacro:include filename="./rover_amalia_chassis.xacro" />
   <model name="rover_amalia_chassis">
-    <xacro:rover_amalia_chassis Ox="0" Oy="0" Oz="0" body_size_x="0.492" body_size_y="0.334" body_size_z="0.1" turret_base_x="0.195" turret_base_y="0"/>
+    <xacro:rover_amalia_chassis Ox="0" Oy="0" Oz="0" body_size_x="0.492" body_size_y="0.334" body_size_z="0.215" turret_base_x="0.195" turret_base_y="0.05"/>
     <pose>0 0 0 0 0 0</pose>
   </model>

File: definitions/rover_amalia_chassis/rover_amalia_chassis.xacro (robot description, xacro)
@@ -33,7 +33,7 @@
         <pose>0 0 0 0 0 0</pose>
         <geometry>
-          <box>
-            <xacro:insert_block name="rover_amalia_chassis_body_size"/>
-          </box>
+          <mesh>
+            <uri>model://rover_amalia_chassis/meshes/chassis.dae</uri>
+          </mesh>
         </geometry>
       </visual>

File: definitions/rover_amalia_leg/model.xacro (robot description, xacro)
@@ -4,5 +4,5 @@
   <model name="rover_amalia_leg">
     <pose>0 0 0 0 0 0</pose>
-    <xacro:rover_amalia_leg Ox="0" Oy="0" Oz="0" prefix="f_r" reflect_xz="1" reflect_yz="1" bar_length="0.2" bar_radius="0.008" wheel_radius="0.08" wheel_length="0.07"/>
+    <xacro:rover_amalia_leg Ox="0" Oy="0" Oz="0" prefix="f_r" reflect_xz="1" reflect_yz="1" bar_length="0.2" bar_radius="0.008" wheel_radius="0.08" wheel_length="0.07" model_root="rover_amalia_leg"/>
   </model>
 </sdf>

File: definitions/rover_amalia_leg/rover_amalia_leg.xacro (robot description, xacro)
@@ -3,5 +3,5 @@
   <xacro:property name="pi" value="3.1415926" />
   <xacro:property name="rover_amalia_leg_bar_z" value="${wheel_radius+bar_length/2}" />
-  <xacro:macro name="rover_amalia_leg" params="Ox Oy Oz prefix reflect_xz reflect_yz bar_length bar_radius wheel_radius wheel_length">
+  <xacro:macro name="rover_amalia_leg" params="Ox Oy Oz prefix reflect_xz reflect_yz bar_length bar_radius wheel_radius wheel_length model_root">
     <link name="rover_amalia_leg_bar_${prefix}">
       <pose>${Ox*reflect_yz} ${Oy*reflect_xz} ${Oz+rover_amalia_leg_bar_z} 0 0 0</pose>
@@ -59,10 +59,9 @@
     </collision>
     <visual name="rover_amalia_leg_wheel_${prefix}_visual">
-      <pose>0 0 0 ${pi/2} 0 0</pose>
+      <pose>0 0 0 0 0 0</pose>
       <geometry>
-        <cylinder>
-          <length>${wheel_length}</length>
-          <radius>${wheel_radius}</radius>
-        </cylinder>
+        <mesh>
+          <uri>model://${model_root}/meshes/wheel.dae</uri>
+        </mesh>
       </geometry>
     </visual>

File: definitions/rover_amalia_turret/rover_amalia_turret.xacro (robot description, xacro)
@@ -72,9 +72,9 @@
       </inertial>
       <visual name="rover_amalia_turret_pan_base_visual">
-        <pose>0 0 0 0 0 0</pose>
-        <geometry>
-          <box>
-            <xacro:insert_block name="rover_amalia_turret_pan_base_size"/>
-          </box>
+        <pose>-0.016 -0.02 0.015 0 0 0</pose>
+        <geometry>
+          <mesh>
+            <uri>model://rover_amalia_turret/meshes/pantilt_pan.dae</uri>
+          </mesh>
         </geometry>
       </visual>
@@ -123,15 +123,15 @@
         <pose>0 0 0 0 0 0</pose>
         <geometry>
-          <box>
-            <xacro:insert_block name="rover_amalia_turret_tilt_base_size"/>
-          </box>
+          <mesh>
+            <uri>model://rover_amalia_turret/meshes/pantilt_tilt.dae</uri>
+          </mesh>
         </geometry>
       </visual>
       <visual name="rover_amalia_turret_camera_set_visual">
-        <pose>0 0 0.03 0 0 0</pose>
-        <geometry>
-          <box>
-            <size>0.02 0.08 0.02</size>
-          </box>
+        <pose>0 0 0.052 0 0 0</pose>
+        <geometry>
+          <mesh>
+            <uri>model://rover_amalia_turret/meshes/pantilt_payload.dae</uri>
+          </mesh>
         </geometry>
       </visual>

Commit message: add pantilt control

File: definitions/rover_amalia/model.xacro (robot description, xacro)
@@ -6,5 +6,5 @@
   <xacro:property name="leg_bar_length" value="0.22"/>
   <xacro:property name="leg_bar_radius" value="0.008"/>
-  <xacro:property name="wheel_radius" value="0.08"/>
+  <xacro:property name="wheel_radius" value="0.09"/>
   <xacro:property name="wheel_length" value="0.07"/>
   <xacro:property name="turret_base_x" value="0.195"/>
@@ -12,6 +12,8 @@
   <xacro:property name="chassis_size_y" value="0.334"/>
   <xacro:property name="chassis_size_z" value="0.215"/>
-  <xacro:property name="chassis_height" value="${leg_bar_length+wheel_radius+0.05}"/>
-  <xacro:property name="leg_x" value="${chassis_size_x*0.27}"/>
+  <xacro:property name="chassis_height" value="${leg_bar_length+wheel_radius+0.02}"/>
+  <xacro:property name="leg_bar_angle" value="${pi/4}"/>
+  <!--use sin function when available-->
+  <xacro:property name="leg_x" value="${chassis_size_x*0.43}"/>
   <xacro:property name="leg_y" value="${chassis_size_y/2 + leg_bar_radius}"/>
   <xacro:macro name="rover_amalia_joint_chassis_leg" params="prefix reflect_xz reflect_yz">
@@ -22,6 +24,6 @@
         <xyz>0 1 0</xyz>
         <limit>
-          <lower>-1e-16</lower>
-          <upper>1e-16</upper>
+          <lower>${-reflect_yz*leg_bar_angle - 1e-4}</lower>
+          <upper>${-reflect_yz*leg_bar_angle + 1e-4}</upper>
         </limit>
         <dynamics/>

File: definitions/rover_amalia_chassis/rover_amalia_chassis.xacro (robot description, xacro)
@@ -19,6 +19,5 @@
       <inertial>
         <pose>0.0216667 0 -0.0215556 0 -0 0</pose>
-        <!--temporary set the mass to 1000, change when all the inertial will be ok-->
-        <mass>100</mass>
+        <mass>30</mass>
         <inertia>
           <ixx>900.12</ixx>

File: definitions/rover_amalia_leg/rover_amalia_leg.xacro (robot description, xacro)
@@ -38,5 +38,5 @@
     <inertial>
       <pose>0 0 0 0 0 0</pose>
-      <mass>1</mass>
+      <mass>5</mass>
       <inertia>
         <ixx>100</ixx>

File: definitions/rover_amalia_turret/rover_amalia_turret.xacro (robot description, xacro)
@@ -226,8 +226,8 @@
       <parent>rover_amalia_turret_bar</parent>
       <axis>
-        <xyz>0 0 1</xyz>
+        <xyz>0 0 -1</xyz>
         <limit>
-          <lower>-1e-16</lower>
-          <upper>1e-16</upper>
+          <lower>-${pi}</lower>
+          <upper>${pi}</upper>
         </limit>
         <dynamics/>
@@ -238,12 +238,18 @@
       <parent>rover_amalia_turret_pan_base</parent>
       <axis>
-        <xyz>0 1 0</xyz>
+        <xyz>0 -1 0</xyz>
         <limit>
-          <lower>-1e-16</lower>
-          <upper>1e-16</upper>
+          <lower>-${pi*3/4</lower>
+          <upper>${pi*3/4</upper>
         </limit>
         <dynamics/>
       </axis>
     </joint>
+    <plugin filename="libgazebo_ros_joint_commander.so" name="joint_commander">
+      <robotNamespace>amalia_rover</robotNamespace>
+      <jointSet1>/ptu/cmd</jointSet1>
+      <jointSet1Joint1>rover_amalia_turret_pan</jointSet1Joint1>
+      <jointSet1Joint2>rover_amalia_turret_tilt</jointSet1Joint2>
+    </plugin>
   </xacro:macro>
 </robot>

Commit message: add .dae files

File: definitions/rover_amalia/model.xacro (robot description, xacro)
@@ -12,23 +12,31 @@
   <xacro:property name="chassis_size_y" value="0.334"/>
   <xacro:property name="chassis_size_z" value="0.215"/>
-  <xacro:property name="chassis_height" value="${leg_bar_length+wheel_radius+0.02}"/>
+  <xacro:property name="chassis_height" value="${leg_bar_length+wheel_radius+0.054}"/>
   <xacro:property name="leg_bar_angle" value="${pi/4}"/>
   <!--use sin function when available-->
-  <xacro:property name="leg_x" value="${chassis_size_x*0.43}"/>
+  <xacro:property name="leg_x" value="${chassis_size_x*0.28}"/>
   <xacro:property name="leg_y" value="${chassis_size_y/2 + leg_bar_radius}"/>
-  <xacro:macro name="rover_amalia_joint_chassis_leg" params="prefix reflect_xz reflect_yz">
+  <xacro:macro name="rover_amalia_joint_chassis_leg" params="prefix reflect_xz reflect_yz index">
     <joint name="rover_amalia_joint_chassis_leg_${prefix}" type="revolute">
+      <pose>0 0 ${leg_bar_length/2} 0 0 0</pose>
       <child>rover_amalia_leg_bar_${prefix}</child>
       <parent>rover_amalia_chassis</parent>
       <axis>
         <xyz>0 1 0</xyz>
-        <limit>
-          <lower>${-reflect_yz*leg_bar_angle - 1e-4}</lower>
-          <upper>${-reflect_yz*leg_bar_angle + 1e-4}</upper>
-        </limit>
         <dynamics/>
         <use_parent_model_frame>1</use_parent_model_frame>
       </axis>
+      <physics>
+        <ode>
+          <provide_feedback>1</provide_feedback>
+        </ode>
+      </physics>
     </joint>
+    <plugin filename="libgazebo_ros_dynamixel_motor.so" name="dynamixel_motor">
+      <joint>rover_amalia_joint_chassis_leg_${prefix}</joint>
+      <base_topic_name>motore_${index}_controller</base_topic_name>
+      <default_pos>0.0</default_pos>
+      <default_torque_limit>100000</default_torque_limit>
+    </plugin>
   </xacro:macro>
   <model name="rover_amalia">
@@ -43,8 +51,8 @@
     <xacro:rover_amalia_leg Ox="${leg_x}" Oy="${leg_y}" Oz="0" prefix="b_l" reflect_xz="-1" reflect_yz="-1" bar_length="${leg_bar_length}" bar_radius="${leg_bar_radius}" wheel_radius="${wheel_radius}" wheel_length="${wheel_length}" model_root="rover_amalia_leg"/>
     <!--additional joints-->
-    <xacro:rover_amalia_joint_chassis_leg prefix="f_r" reflect_xz="1" reflect_yz="1"/>
-    <xacro:rover_amalia_joint_chassis_leg prefix="f_l" reflect_xz="-1" reflect_yz="1"/>
-    <xacro:rover_amalia_joint_chassis_leg prefix="b_r" reflect_xz="1" reflect_yz="-1"/>
-    <xacro:rover_amalia_joint_chassis_leg prefix="b_l" reflect_xz="-1" reflect_yz="-1"/>
+    <xacro:rover_amalia_joint_chassis_leg prefix="f_r" reflect_xz="1" reflect_yz="1" index="1"/>
+    <xacro:rover_amalia_joint_chassis_leg prefix="f_l" reflect_xz="-1" reflect_yz="1" index="2"/>
+    <xacro:rover_amalia_joint_chassis_leg prefix="b_r" reflect_xz="1" reflect_yz="-1" index="3"/>
+    <xacro:rover_amalia_joint_chassis_leg prefix="b_l" reflect_xz="-1" reflect_yz="-1" index="4"/>
     <joint name="rover_amalia_joint_turret_base_turret" type="revolute">
       <child>rover_amalia_turret_bar</child>

File: definitions/rover_amalia_chassis/rover_amalia_chassis.xacro (robot description, xacro)
@@ -20,12 +20,12 @@
         <pose>0.0216667 0 -0.0215556 0 -0 0</pose>
         <mass>30</mass>
-        <inertia>
-          <ixx>900.12</ixx>
-          <ixy>-3.46945e-18</ixy>
-          <ixz>-0.0139533</ixz>
-          <iyy>900.352</iyy>
-          <iyz>0</iyz>
-          <izz>900.455</izz>
-        </inertia>
+        <!--<inertia>-->
+          <!--<ixx>900.12</ixx>-->
+          <!--<ixy>-3.46945e-18</ixy>-->
+          <!--<ixz>-0.0139533</ixz>-->
+          <!--<iyy>900.352</iyy>-->
+          <!--<iyz>0</iyz>-->
+          <!--<izz>900.455</izz>-->
+        <!--</inertia>-->
       </inertial>
       <visual name="rover_amalia_chassis_body_visual">

File: definitions/rover_amalia_leg/rover_amalia_leg.xacro (robot description, xacro)
@@ -35,5 +35,5 @@
   </link>
   <link name="rover_amalia_leg_wheel_${prefix}">
-    <pose>${Ox*reflect_yz} ${(Oy+wheel_length/2+bar_radius+0.001)*reflect_xz} ${wheel_radius} 0 0 0</pose>
+    <pose>${Ox*reflect_yz} ${(Oy+wheel_length/2+bar_radius+0.001)*reflect_xz} ${Oz + wheel_radius} 0 0 0</pose>
     <inertial>
       <pose>0 0 0 0 0 0</pose>

File: definitions/rover_amalia_turret/rover_amalia_turret.xacro (robot description, xacro)
@@ -20,4 +20,5 @@
     <size>0.06 0.02 ${rover_amalia_turret_pan_tilt_height}</size>
   </xacro:property>
+  <xacro:property name="rover_amalia_turret_robot_namespace" value="rover_amalia" />
   <xacro:macro name="rover_amalia_turret" params="Ox Oy Oz bar_height">
     <link name="rover_amalia_turret_bar">
@@ -137,5 +138,5 @@
       </visual>
       <sensor name="depth_camera" type="depth">
-        <pose>0 0 0 0 ${pi} 0</pose>
+        <pose>0 0 0 0 0 0</pose>
         <camera>
           <horizontal_fov>1.578</horizontal_fov>
@@ -152,4 +153,5 @@
         <plugin filename="libgazebo_ros_depth_camera.so" name="depth_camera_plugin">
           <alwaysOn>1</alwaysOn>
+          <robotNamespace>${rover_amalia_turret_robot_namespace}</robotNamespace>
           <updateRate>10.0</updateRate>
           <imageTopicName>image_raw</imageTopicName>
@@ -175,5 +177,5 @@
         <visualize>true</visualize>
         <camera name="left">
-          <pose>0 0 0 0 3.14 0</pose>
+          <pose>0 0 0 0 0 0</pose>
           <horizontal_fov>1.047</horizontal_fov>
           <image>
@@ -187,5 +189,5 @@
         </camera>
         <camera name="right">
-          <pose>0 -0.2 0 0 3.14 0</pose>
+          <pose>0 0 0 0 0 0</pose>
           <horizontal_fov>1.047</horizontal_fov>
           <image>
@@ -240,6 +242,6 @@
         <xyz>0 -1 0</xyz>
         <limit>
-          <lower>-${pi*3/4</lower>
-          <upper>${pi*3/4</upper>
+          <lower>${-pi*3/4}</lower>
+          <upper>${pi*3/4}</upper>
         </limit>
         <dynamics/>
@@ -247,5 +249,5 @@
     </joint>
     <plugin filename="libgazebo_ros_joint_commander.so" name="joint_commander">
-      <robotNamespace>amalia_rover</robotNamespace>
+      <robotNamespace>${rover_amalia_turret_robot_namespace}</robotNamespace>
       <jointSet1>/ptu/cmd</jointSet1>
       <jointSet1Joint1>rover_amalia_turret_pan</jointSet1Joint1>

Commit message: add joint publishers

File: definitions/rover_amalia/model.xacro (robot description, xacro)
@@ -24,5 +24,9 @@
       <axis>
         <xyz>0 1 0</xyz>
-        <dynamics/>
+        <!--<dynamics>-->
+          <!--<damping>0.0001</damping>-->
+          <!--<spring_stiffness>1</spring_stiffness>-->
+          <!--<spring_reference>0</spring_reference>-->
+        <!--</dynamics>-->
         <use_parent_model_frame>1</use_parent_model_frame>
       </axis>
@@ -37,7 +41,10 @@
       <joint>rover_amalia_joint_chassis_leg_${prefix}</joint>
       <base_topic_name>motore_${index}_controller</base_topic_name>
-      <default_pos>0.0</default_pos>
+      <default_pos>${-2*reflect_yz}</default_pos>
       <default_torque_limit>100000</default_torque_limit>
       <reduction_value>6.3</reduction_value>
+    </plugin>
+    <plugin filename="libgazebo_ros_joint_state_publisher.so" name="arm_${prefix}">
+      <jointName>rover_amalia_joint_chassis_leg_${prefix}</jointName>
     </plugin>
   </xacro:macro>

File: definitions/rover_amalia_leg/rover_amalia_leg.xacro (robot description, xacro)
@@ -86,12 +86,15 @@
       <parent>rover_amalia_leg_bar_${prefix}</parent>
       <axis>
-	<xyz>0 1 0</xyz>
-	<limit>
+        <xyz>0 1 0</xyz>
+        <limit>
           <lower>-1e+16</lower>
           <upper>1e+16</upper>
-	</limit>
-	<use_parent_model_frame>1</use_parent_model_frame>
+        </limit>
+        <use_parent_model_frame>1</use_parent_model_frame>
       </axis>
     </joint>
+    <plugin filename="libgazebo_ros_joint_state_publisher.so" name="wheel_${prefix}">
+      <jointName>rover_amalia_leg_shaft_${prefix}</jointName>
+    </plugin>
   </xacro:macro>
 </robot>

File: definitions/rover_amalia_turret/rover_amalia_turret.xacro (robot description, xacro)
@@ -254,4 +254,10 @@
       <jointSet1Joint2>rover_amalia_turret_tilt</jointSet1Joint2>
     </plugin>
+    <plugin filename="libgazebo_ros_joint_state_publisher.so" name="pan">
+      <jointName>rover_amalia_turret_pan</jointName>
+    </plugin>
+    <plugin filename="libgazebo_ros_joint_state_publisher.so" name="tilt">
+      <jointName>rover_amalia_turret_tilt</jointName>
+    </plugin>
   </xacro:macro>
 </robot>
