Commit message: add ramp1 and ramp2

File: definitions/rover_amalia/model.xacro (robot description, xacro)
@@ -47,4 +47,5 @@
     <plugin filename="libgazebo_ros_joint_state_publisher.so" name="arm_${prefix}">
       <jointName>rover_amalia_joint_chassis_leg_${prefix}</jointName>
+      <updateRate>30</updateRate>
     </plugin>
   </xacro:macro>

File: definitions/rover_amalia_leg/rover_amalia_leg.xacro (robot description, xacro)
@@ -96,4 +96,5 @@
     <plugin filename="libgazebo_ros_joint_state_publisher.so" name="wheel_${prefix}">
       <jointName>rover_amalia_leg_shaft_${prefix}</jointName>
+      <updateRate>30</updateRate>
     </plugin>
   </xacro:macro>

File: definitions/rover_amalia_leg_test_bench/model.xacro (robot description, xacro)
@@ -92,4 +92,5 @@
           <provide_feedback>1</provide_feedback>
         </ode>
+        <provide_feedback>1</provide_feedback>
       </physics>
     </joint>

File: definitions/rover_amalia_turret/rover_amalia_turret.xacro (robot description, xacro)
@@ -6,17 +6,17 @@
     <pose>${Ox} ${Oy} ${Oz} 0 0 0</pose>
   </xacro:property>
-  <xacro:property name="rover_amalia_turret_pan_base_height" value="0.02"/>
-  <xacro:property name="rover_amalia_turret_pan_base_pose">
-    <pose>${Ox} ${Oy} ${Oz+bar_height+rover_amalia_turret_pan_base_height/2} 0 0 0</pose>
-  </xacro:property>
-  <xacro:property name="rover_amalia_turret_pan_base_size">
-      <size>0.04 0.06 ${rover_amalia_turret_pan_base_height} </size>
+  <xacro:property name="rover_amalia_turret_tilt_base_height" value="0.02"/>
+  <xacro:property name="rover_amalia_turret_tilt_base_pose">
+    <pose>${Ox} ${Oy} ${Oz+bar_height+rover_amalia_turret_tilt_base_height/2} 0 0 0</pose>
+  </xacro:property>
+  <xacro:property name="rover_amalia_turret_tilt_base_size">
+      <size>0.09 0.03 0.05 </size>
   </xacro:property>
   <xacro:property name="rover_amalia_turret_pan_tilt_height" value="0.04"/>
-  <xacro:property name="rover_amalia_turret_tilt_base_pose">
-    <pose>${Ox} ${Oy-0.01} ${Oz+bar_height+rover_amalia_turret_pan_base_height+rover_amalia_turret_pan_tilt_height/2} 0 0 0</pose>
-  </xacro:property>
-  <xacro:property name="rover_amalia_turret_tilt_base_size">
-    <size>0.06 0.02 ${rover_amalia_turret_pan_tilt_height}</size>
+  <xacro:property name="rover_amalia_turret_tilt_hinge_pose">
+    <pose>${Ox} ${Oy-0.01} ${Oz+bar_height+rover_amalia_turret_tilt_base_height+rover_amalia_turret_pan_tilt_height/2} 0 0 0</pose>
+  </xacro:property>
+  <xacro:property name="rover_amalia_turret_tilt_hinge_size">
+    <size>0.03 0.07 ${rover_amalia_turret_pan_tilt_height}</size>
   </xacro:property>
   <xacro:property name="rover_amalia_turret_robot_namespace" value="rover_amalia" />
@@ -24,16 +24,16 @@
     <link name="rover_amalia_turret_bar">
       <xacro:insert_block name="rover_amalia_turret_bar_pose"/>
-      <inertial>
-        <pose>0 0 0 0 0 0</pose>
-        <mass>0.5</mass>
-        <inertia>
-          <ixx>0.001</ixx>
-          <ixy>0</ixy>
-          <ixz>0</ixz>
-          <iyy>0.001</iyy>
-          <iyz>0</iyz>
-          <izz>0.001</izz>
-        </inertia>
-      </inertial>
+      <!--<inertial>-->
+        <!--<pose>0 0 0 0 0 0</pose>-->
+        <!--<mass>0.78</mass>-->
+        <!--<inertia>-->
+          <!--<ixx>0.00000027555</ixx>-->
+          <!--<ixy>0</ixy>-->
+          <!--<ixz>0</ixz>-->
+          <!--<iyy>0.00000027555</iyy>-->
+          <!--<iyz>0</iyz>-->
+          <!--<izz>0.00000027755</izz>-->
+        <!--</inertia>-->
+      <!--</inertial>-->
       <collision name="rover_amalia_turret_bar_collision">
         <pose>0 0 ${bar_height/2} 0 0 0</pose>
@@ -58,19 +58,34 @@
       <gravity>1</gravity>
     </link>
-    <link name="rover_amalia_turret_pan_base">
-      <xacro:insert_block name="rover_amalia_turret_pan_base_pose"/>
-      <inertial>
-        <pose>0 0 0 0 0 0</pose>
-        <mass>1</mass>
-        <inertia>
-          <ixx>0.001</ixx>
-          <ixy>0</ixy>
-          <ixz>0</ixz>
-          <iyy>0.00100</iyy>
-          <iyz>0</iyz>
-          <izz>0.00100</izz>
-        </inertia>
-      </inertial>
-      <visual name="rover_amalia_turret_pan_base_visual">
+    <link name="rover_amalia_turret_tilt_base">
+      <xacro:insert_block name="rover_amalia_turret_tilt_base_pose"/>
+      <!--correct inertial for pan base, use later-->
+      <!--<inertial>-->
+        <!--<pose>-0.00699 0.17952 0.02755 0 0 0</pose>-->
+        <!--<mass>0.22386</mass>-->
+        <!--<inertia>-->
+          <!--<ixx>0.00010575745</ixx>-->
+          <!--<ixy>0.00002524815</ixy>-->
+          <!--<ixz>0</ixz>-->
+          <!--<iyy>0.00100</iyy>-->
+          <!--<iyz>0</iyz>-->
+          <!--<izz>0.00021796864</izz>-->
+        <!--</inertia>-->
+      <!--</inertial>-->
+      <!--this are ok, leave them:-->
+      <!--<inertial>-->
+        <!--<pose>0.012 -0.21853 0.02754  0 0 0</pose>-->
+        <!--<pose>0 0 0 0 0 0</pose>-->
+        <!--<mass>0.02786</mass>-->
+        <!--<inertia>-->
+          <!--<ixx>0.00002247622</ixx>-->
+          <!--<ixy>0.</ixy>-->
+          <!--<ixz>0</ixz>-->
+          <!--<iyy>0.00001850151</iyy>-->
+          <!--<iyz>0</iyz>-->
+          <!--<izz>0.00000707185</izz>-->
+        <!--</inertia>-->
+      <!--</inertial>-->
+      <visual name="rover_amalia_turret_tilt_base_visual">
         <pose>-0.016 -0.02 0.015 0 0 0</pose>
         <geometry>
@@ -80,4 +95,13 @@
         </geometry>
       </visual>
+      <collision name="rover_amalia_turret_tilt_base_collision">
+        <pose>-0.02 0 0.01 0 0 0</pose>
+        <xacro:insert_block name="rover_amalia_turret_tilt_hinge_pose"/>
+        <geometry>
+          <box>
+            <xacro:insert_block name="rover_amalia_turret_tilt_base_size"/>
+          </box>
+        </geometry>
+      </collision>
       <velocity_decay>
         <linear>0</linear>
@@ -88,24 +112,12 @@
       <gravity>1</gravity>
     </link>
-    <link name="rover_amalia_turret_tilt_base">
-      <xacro:insert_block name="rover_amalia_turret_tilt_base_pose"/>
-      <inertial>
+    <link name="rover_amalia_turret_tilt_hinge">
+      <xacro:insert_block name="rover_amalia_turret_tilt_hinge_pose"/>
+      <collision name="rover_amalia_turret_tilt_hinge_collision">
         <pose>0 0 0 0 0 0</pose>
-        <mass>2</mass>
-        <inertia>
-          <ixx>0.00200001</ixx>
-          <ixy>0</ixy>
-          <ixz>0</ixz>
-          <iyy>0.00200001</iyy>
-          <iyz>0</iyz>
-          <izz>0.00200</izz>
-        </inertia>
-      </inertial>
-      <collision name="rover_amalia_turret_tilt_base_collision">
-        <pose>0 0 0 0 0 0</pose>
-        <xacro:insert_block name="rover_amalia_turret_tilt_base_pose"/>
+        <xacro:insert_block name="rover_amalia_turret_tilt_hinge_pose"/>
         <geometry>
           <box>
-            <xacro:insert_block name="rover_amalia_turret_tilt_base_size"/>
+            <xacro:insert_block name="rover_amalia_turret_tilt_hinge_size"/>
           </box>
         </geometry>
@@ -121,5 +133,5 @@
         </surface>
       </collision>
-      <visual name="rover_amalia_turret_tilt_base_visual">
+      <visual name="rover_amalia_turret_tilt_hinge_visual">
         <pose>0 0 0 0 0 0</pose>
         <geometry>
@@ -203,9 +215,9 @@
           <alwaysOn>true</alwaysOn>
           <updateRate>60.0</updateRate>
-          <cameraName>camera</cameraName>
+          <cameraName>stereo</cameraName>
           <imageTopicName>image_raw</imageTopicName>
           <cameraInfoTopicName>camera_info</cameraInfoTopicName>
           <frameName>left_camera_optical_frame</frameName>
-          <!--<rightFrameName>right_camera_optical_frame</rightFrameName>-->
+          <rightFrameName>right_camera_optical_frame</rightFrameName>
           <hackBaseline>0.07</hackBaseline>
           <distortionK1>0.0</distortionK1>
@@ -225,5 +237,5 @@
     </link>
     <joint name="rover_amalia_turret_pan" type="revolute">
-      <child>rover_amalia_turret_pan_base</child>
+      <child>rover_amalia_turret_tilt_base</child>
       <parent>rover_amalia_turret_bar</parent>
       <axis>
@@ -233,10 +245,15 @@
           <upper>${pi}</upper>
         </limit>
-        <dynamics/>
       </axis>
+      <physics>
+        <ode>
+          <cfm>0.0001</cfm>
+          <erp>0.2</erp>
+        </ode>
+      </physics>
     </joint>
     <joint name="rover_amalia_turret_tilt" type="revolute">
-      <child>rover_amalia_turret_tilt_base</child>
-      <parent>rover_amalia_turret_pan_base</parent>
+      <child>rover_amalia_turret_tilt_hinge</child>
+      <parent>rover_amalia_turret_tilt_base</parent>
       <axis>
         <xyz>0 -1 0</xyz>
@@ -245,6 +262,11 @@
           <upper>${pi*3/4}</upper>
         </limit>
-        <dynamics/>
       </axis>
+      <physics>
+        <ode>
+          <cfm>0</cfm>
+          <erp>0.2</erp>
+        </ode>
+      </physics>
     </joint>
     <plugin filename="libgazebo_ros_joint_commander.so" name="joint_commander">
@@ -256,7 +278,9 @@
     <plugin filename="libgazebo_ros_joint_state_publisher.so" name="pan">
       <jointName>rover_amalia_turret_pan</jointName>
+      <updateRate>30</updateRate>
     </plugin>
     <plugin filename="libgazebo_ros_joint_state_publisher.so" name="tilt">
       <jointName>rover_amalia_turret_tilt</jointName>
+      <updateRate>30</updateRate>
     </plugin>
   </xacro:macro>

Commit message: add joint velocities

File: definitions/rover_amalia/model.xacro (robot description, xacro)
@@ -24,4 +24,10 @@
       <axis>
         <xyz>0 1 0</xyz>
+        <limit>
+          <lower>${-pi}</lower>
+          <upper>${pi}</upper>
+          <effort>1000</effort>
+          <velocity>1000</velocity>
+        </limit>
         <!--<dynamics>-->
           <!--<damping>0.0001</damping>-->
@@ -46,4 +52,5 @@
     </plugin>
     <plugin filename="libgazebo_ros_joint_state_publisher.so" name="arm_${prefix}">
+      <robotNamespace></robotNamespace>
       <jointName>rover_amalia_joint_chassis_leg_${prefix}</jointName>
       <updateRate>30</updateRate>
@@ -73,4 +80,6 @@
           <lower>-1e-16</lower>
           <upper>1e-16</upper>
+          <effort>1000</effort>
+          <velocity>1000</velocity>
         </limit>
         <dynamics/>

File: definitions/rover_amalia_leg/rover_amalia_leg.xacro (robot description, xacro)
@@ -90,4 +90,6 @@
           <lower>-1e+16</lower>
           <upper>1e+16</upper>
+          <effort>1000</effort>
+          <velocity>1000</velocity>
         </limit>
         <use_parent_model_frame>1</use_parent_model_frame>
@@ -95,4 +97,5 @@
     </joint>
     <plugin filename="libgazebo_ros_joint_state_publisher.so" name="wheel_${prefix}">
+      <robotNamespace></robotNamespace>
       <jointName>rover_amalia_leg_shaft_${prefix}</jointName>
       <updateRate>30</updateRate>

File: definitions/rover_amalia_turret/rover_amalia_turret.xacro (robot description, xacro)
@@ -244,4 +244,6 @@
           <lower>-${pi}</lower>
           <upper>${pi}</upper>
+          <effort>1000</effort>
+          <velocity>1000</velocity>
         </limit>
       </axis>
@@ -261,4 +263,6 @@
           <lower>${-pi*3/4}</lower>
           <upper>${pi*3/4}</upper>
+          <effort>1000</effort>
+          <velocity>1000</velocity>
         </limit>
       </axis>
@@ -277,8 +281,10 @@
     </plugin>
     <plugin filename="libgazebo_ros_joint_state_publisher.so" name="pan">
+      <robotNamespace></robotNamespace>
       <jointName>rover_amalia_turret_pan</jointName>
       <updateRate>30</updateRate>
     </plugin>
     <plugin filename="libgazebo_ros_joint_state_publisher.so" name="tilt">
+      <robotNamespace></robotNamespace>
       <jointName>rover_amalia_turret_tilt</jointName>
       <updateRate>30</updateRate>

Commit message: fix link positions

File: definitions/rover_amalia/model.xacro (robot description, xacro)
@@ -62,5 +62,5 @@
     <!--main components-->
     <xacro:rover_amalia_turret Ox="${turret_base_x}" Oy="0" Oz="${chassis_height+0.1}" bar_height="0.2"/>
-    <xacro:rover_amalia_chassis Ox="0" Oy="0" Oz="${chassis_height}" body_size_x="${chassis_size_x}" body_size_y="${chassis_size_y}" body_size_z="${chassis_size_z}" turret_base_x="${turret_base_x}" turret_base_y="0.05"/>
+    <xacro:rover_amalia_chassis Ox="0" Oy="0" Oz="${chassis_height}" body_size_x="${chassis_size_x}" body_size_y="${chassis_size_y}" body_size_z="${chassis_size_z}" turret_base_x="${turret_base_x}" turret_base_y="0"/>
     <xacro:rover_amalia_leg Ox="${leg_x}" Oy="${leg_y}" Oz="0" prefix="f_r" reflect_xz="1" reflect_yz="1" bar_length="${leg_bar_length}" bar_radius="${leg_bar_radius}" wheel_radius="${wheel_radius}" wheel_length="${wheel_length}" model_root="rover_amalia_leg"/>
     <xacro:rover_amalia_leg Ox="${leg_x}" Oy="${leg_y}" Oz="0" prefix="f_l" reflect_xz="-1" reflect_yz="1" bar_length="${leg_bar_length}" bar_radius="${leg_bar_radius}" wheel_radius="${wheel_radius}" wheel_length="${wheel_length}" model_root="rover_amalia_leg"/>

File: definitions/rover_amalia_chassis/model.xacro (robot description, xacro)
@@ -3,5 +3,5 @@
   <xacro:include filename="./rover_amalia_chassis.xacro" />
   <model name="rover_amalia_chassis">
-    <xacro:rover_amalia_chassis Ox="0" Oy="0" Oz="0" body_size_x="0.492" body_size_y="0.334" body_size_z="0.215" turret_base_x="0.195" turret_base_y="0.05"/>
+    <xacro:rover_amalia_chassis Ox="0" Oy="0" Oz="0" body_size_x="0.492" body_size_y="0.334" body_size_z="0.215" turret_base_x="0.195" turret_base_y="0"/>
     <pose>0 0 0 0 0 0</pose>
   </model>

File: definitions/rover_amalia_chassis/rover_amalia_chassis.xacro (robot description, xacro)
@@ -13,5 +13,5 @@
     <size>${rover_amalia_chassis_rangefinder_size_y} 0.03 ${rover_amalia_chassis_rangefinder_size_y}</size>
   </xacro:property>
-  <xacro:property name="rover_amalia_chassis_turret_base_z" value="0.073" />
+  <xacro:property name="rover_amalia_chassis_turret_base_z" value="0.12" />
   <xacro:macro name="rover_amalia_chassis" params="Ox Oy Oz body_size_x body_size_y body_size_z turret_base_x turret_base_y">
     <link name="rover_amalia_chassis">

File: definitions/rover_amalia_turret/rover_amalia_turret.xacro (robot description, xacro)
@@ -19,5 +19,5 @@
   <xacro:property name="rover_amalia_turret_pan_tilt_height" value="0.04"/>
   <xacro:property name="rover_amalia_turret_tilt_hinge_pose">
-    <pose>${Ox} ${Oy-0.01} ${Oz+pan_base_height+bar_height+rover_amalia_turret_tilt_base_height+rover_amalia_turret_pan_tilt_height/2} 0 0 0</pose>
+    <pose>${Ox} ${Oy} ${Oz+pan_base_height+bar_height+rover_amalia_turret_tilt_base_height+rover_amalia_turret_pan_tilt_height/2} 0 0 0</pose>
   </xacro:property>
   <xacro:property name="rover_amalia_turret_tilt_hinge_size">

Commit message: add another inertial dummy

File: definitions/rover_amalia/model.xacro (robot description, xacro)
@@ -4,4 +4,5 @@
   <xacro:include filename="../rover_amalia_chassis/rover_amalia_chassis.xacro"/>
   <xacro:include filename="../rover_amalia_turret/rover_amalia_turret.xacro"/>
+  <xacro:include filename="../rover_amalia_turret_inertials/rover_amalia_turret_inertials.xacro" />
   <xacro:property name="leg_bar_length" value="0.22"/>
   <xacro:property name="leg_bar_radius" value="0.008"/>
@@ -62,4 +63,5 @@
     <!--main components-->
     <xacro:rover_amalia_turret Ox="${turret_base_x}" Oy="0" Oz="${chassis_height+0.1}" bar_height="0.2"/>
+    <xacro:rover_amalia_turret_inertials Ox="${turret_base_x}" Oy="0" Oz="${chassis_height+0.1}" bar_height="0.2"/>
     <xacro:rover_amalia_chassis Ox="0" Oy="0" Oz="${chassis_height}" body_size_x="${chassis_size_x}" body_size_y="${chassis_size_y}" body_size_z="${chassis_size_z}" turret_base_x="${turret_base_x}" turret_base_y="0"/>
     <xacro:rover_amalia_leg Ox="${leg_x}" Oy="${leg_y}" Oz="0" prefix="f_r" reflect_xz="1" reflect_yz="1" bar_length="${leg_bar_length}" bar_radius="${leg_bar_radius}" wheel_radius="${wheel_radius}" wheel_length="${wheel_length}" model_root="rover_amalia_leg"/>
@@ -74,4 +76,34 @@
     <joint name="rover_amalia_joint_turret_base_turret" type="revolute">
       <child>rover_amalia_turret_bar</child>
+      <parent>rover_amalia_chassis</parent>
+      <axis>
+        <xyz>0 0 1</xyz>
+        <limit>
+          <lower>-1e-16</lower>
+          <upper>1e-16</upper>
+          <effort>1000</effort>
+          <velocity>1000</velocity>
+        </limit>
+        <dynamics/>
+        <use_parent_model_frame>1</use_parent_model_frame>
+      </axis>
+    </joint>
+    <joint name="rover_amalia_joint_turret_base_turret_dummy" type="revolute">
+      <child>rover_amalia_turret_bar_inertial_dummy</child>
+      <parent>rover_amalia_chassis</parent>
+      <axis>
+        <xyz>0 0 1</xyz>
+        <limit>
+          <lower>-1e-16</lower>
+          <upper>1e-16</upper>
+          <effort>1000</effort>
+          <velocity>1000</velocity>
+        </limit>
+        <dynamics/>
+        <use_parent_model_frame>1</use_parent_model_frame>
+      </axis>
+    </joint>
+    <joint name="rover_amalia_joint_turret_base_turret_payload_dummy" type="revolute">
+      <child>rover_amalia_turret_payload_inertial_dummy</child>
       <parent>rover_amalia_chassis</parent>
       <axis>

File: definitions/rover_amalia_turret/rover_amalia_turret.xacro (robot description, xacro)
@@ -9,5 +9,5 @@
   <xacro:property name="pan_base_height" value="0.043"/>
   <xacro:property name="rover_amalia_turret_pan_base_pose">
-    <pose>${Ox} ${Oy+0.015} ${Oz+pan_base_height+bar_height+rover_amalia_turret_tilt_base_height/2}-0.01 0 0 0</pose>
+    <pose>${Ox} ${Oy+0.015} ${Oz+pan_base_height+bar_height+rover_amalia_turret_tilt_base_height/2-0.01} 0 0 0</pose>
   </xacro:property>
   <xacro:property name="rover_amalia_turret_tilt_base_pose">
@@ -26,19 +26,4 @@
   <xacro:property name="rover_amalia_turret_robot_namespace" value="rover_amalia" />
   <xacro:macro name="rover_amalia_turret" params="Ox Oy Oz bar_height">
-    <link name="rover_amalia_turret_bar_inertial_dummy">
-      <xacro:insert_block name="rover_amalia_turret_bar_pose"/>
-      <inertial>
-        <pose>0 0 0 0 0 0</pose>
-        <mass>0.78</mass>
-        <inertia>
-          <ixx>0.00000027555</ixx>
-          <ixy>0</ixy>
-          <ixz>0</ixz>
-          <iyy>0.00000027555</iyy>
-          <iyz>0</iyz>
-          <izz>0.00000027755</izz>
-        </inertia>
-      </inertial>
-    </link>
     <link name="rover_amalia_turret_bar">
       <xacro:insert_block name="rover_amalia_turret_bar_pose"/>
@@ -62,34 +47,7 @@
       <self_collide>0</self_collide>
       <kinematic>0</kinematic>
-      <gravity>1</gravity>
-    </link>
-    <link name="rover_amalia_turret_pan_base_inertial_dummy">
-      <xacro:insert_block name="rover_amalia_turret_pan_base_pose"/>
+      <gravity>0</gravity>
       <inertial>
-        <pose>-0.00699 0.17952 0.02755 0 0 0</pose>
-        <mass>0.22386</mass>
-        <inertia>
-          <ixx>0.00010575745</ixx>
-          <ixy>0.00002524815</ixy>
-          <ixz>0</ixz>
-          <iyy>0.00100</iyy>
-          <iyz>0</iyz>
-          <izz>0.00021796864</izz>
-        </inertia>
-      </inertial>
-    </link>
-    <link name="rover_amalia_turret_tilt_base_inertial_dummy">
-      <inertial>
-        <pose>0.012 -0.21853 0.02754  0 0 0</pose>
-        <pose>0 0 0 0 0 0</pose>
-        <mass>0.02786</mass>
-        <inertia>
-          <ixx>0.00002247622</ixx>
-          <ixy>0.</ixy>
-          <ixz>0</ixz>
-          <iyy>0.00001850151</iyy>
-          <iyz>0</iyz>
-          <izz>0.00000707185</izz>
-        </inertia>
+        <mass>0.000001</mass>
       </inertial>
     </link>
@@ -119,5 +77,8 @@
       <self_collide>0</self_collide>
       <kinematic>0</kinematic>
-      <gravity>1</gravity>
+      <gravity>0</gravity>
+      <inertial>
+        <mass>0.000001</mass>
+      </inertial>
     </link>
     <link name="rover_amalia_turret_tilt_hinge">
@@ -243,5 +204,8 @@
       <self_collide>0</self_collide>
       <kinematic>0</kinematic>
-      <gravity>1</gravity>
+      <gravity>0</gravity>
+      <inertial>
+        <mass>0.000001</mass>
+      </inertial>
     </link>
     <joint name="rover_amalia_turret_pan" type="revolute">
@@ -278,5 +242,5 @@
       <physics>
         <ode>
-          <cfm>0</cfm>
+          <cfm>0.0001</cfm>
           <erp>0.2</erp>
         </ode>
