Commit message: fix cameras and meshes

File: definitions/rover_amalia/model.xacro (robot description, xacro)
@@ -17,5 +17,5 @@
   <!--use sin function when available-->
   <xacro:property name="leg_x" value="${chassis_size_x*0.28}"/>
-  <xacro:property name="leg_y" value="${chassis_size_y/2 + leg_bar_radius}"/>
+  <xacro:property name="leg_y" value="${chassis_size_y/2 + leg_bar_radius+0.01}"/>
   <xacro:macro name="rover_amalia_joint_chassis_leg" params="prefix reflect_xz reflect_yz index">
     <joint name="rover_amalia_joint_chassis_leg_${prefix}" type="revolute">

File: definitions/rover_amalia_chassis/rover_amalia_chassis.xacro (robot description, xacro)
@@ -14,4 +14,5 @@
   </xacro:property>
   <xacro:property name="rover_amalia_chassis_turret_base_z" value="0.12" />
+  <xacro:property name="rover_amalia_range_finder_z" value="-0.1" />
   <xacro:macro name="rover_amalia_chassis" params="Ox Oy Oz body_size_x body_size_y body_size_z turret_base_x turret_base_y">
     <link name="rover_amalia_chassis">
@@ -63,6 +64,14 @@
         </geometry>
       </visual>
+      <visual name="rover_amalia_chassis_cpci">
+        <pose>0 -0.08 0.1 0 0 0</pose>
+        <geometry>
+          <mesh>
+            <uri>model://rover_amalia_chassis/meshes/cpci.dae</uri>
+          </mesh>
+        </geometry>
+      </visual>
       <visual name="rover_amalia_chassis_front_up_rangefinder_visual">
-        <pose>0.246 0 -0.05 0 -0 0</pose>
+        <pose>0.246 0 ${rover_amalia_range_finder_z} 0 -0 0</pose>
         <geometry>
           <box>
@@ -72,5 +81,5 @@
       </visual>
       <visual name="rover_amalia_chassis_front_down_rangefinder_visual">
-        <pose>${0.246-rover_amalia_chassis_rangefinder_size_y} 0 ${-0.05-rover_amalia_chassis_rangefinder_size_y} 0 1.57 0</pose>
+        <pose>${0.246-rover_amalia_chassis_rangefinder_size_y} 0 ${rover_amalia_range_finder_z - rover_amalia_chassis_rangefinder_size_y} 0 1.57 0</pose>
         <geometry>
           <box>
@@ -80,5 +89,5 @@
       </visual>
       <sensor name="range_front_down_ray" type="ray">
-          <pose>0.25 0 -0.09 0 ${pi/2} 0</pose>
+          <pose>0.25 0 ${rover_amalia_range_finder_z} 0 ${pi/2} 0</pose>
           <ray>
               <scan>
@@ -96,6 +105,5 @@
               </range>
           </ray>
-          <!-- test plugin -->
-          <plugin name="plugin_1" filename="libgazebo_ros_range_finder.so">
+          <plugin name="range_finder_plugin_front" filename="libgazebo_ros_range_finder.so">
               <gaussianNoise>0.005</gaussianNoise>
               <alwaysOn>true</alwaysOn>
@@ -109,5 +117,5 @@
       </sensor>
       <visual name="rover_amalia_chassis_rear_up_rangefinder_visual">
-        <pose>-0.246 0 -0.05 3.14159 0.00159265 3.14159</pose>
+        <pose>-0.246 0 ${rover_amalia_range_finder_z} 3.14159 0.00159265 3.14159</pose>
         <geometry>
           <box>
@@ -117,5 +125,5 @@
       </visual>
       <visual name="rover_amalia_chassis_rear_down_rangefinder_visual">
-        <pose>${-0.246+rover_amalia_chassis_rangefinder_size_y} 0 ${-0.05-rover_amalia_chassis_rangefinder_size_y} 0 1.57 0</pose>
+        <pose>${-0.246+rover_amalia_chassis_rangefinder_size_y} 0 ${rover_amalia_range_finder_z - rover_amalia_chassis_rangefinder_size_y} 0 1.57 0</pose>
         <geometry>
           <box>
@@ -125,5 +133,5 @@
       </visual>
       <sensor name="range_rear_down_ray" type="ray">
-          <pose>${-0.248+rover_amalia_chassis_rangefinder_size_y} 0 ${-0.05-rover_amalia_chassis_rangefinder_size_y} 0 1.57 0</pose>
+          <pose>${-0.248+rover_amalia_chassis_rangefinder_size_y} 0 ${rover_amalia_range_finder_z - rover_amalia_chassis_rangefinder_size_y} 0 1.57 0</pose>
           <ray>
               <scan>
@@ -141,6 +149,5 @@
               </range>
           </ray>
-          <!-- test plugin -->
-          <plugin name="plugin_1" filename="libgazebo_ros_range_finder.so">
+          <plugin name="range_finder_plugin_rear" filename="libgazebo_ros_range_finder.so">
               <gaussianNoise>0.005</gaussianNoise>
               <alwaysOn>true</alwaysOn>

File: definitions/rover_amalia_leg/rover_amalia_leg.xacro (robot description, xacro)
@@ -7,74 +7,64 @@
       <pose>${Ox*reflect_yz} ${Oy*reflect_xz} ${Oz+rover_amalia_leg_bar_z} 0 0 0</pose>
       <inertial>
-	<pose>0 0 0 0 0 0</pose>
-	<mass>0.31</mass>
-	<inertia>
-          <ixx>0.00279048</ixx>
-          <ixy>0</ixy>
-          <ixz>-0.00003956</ixz>
-          <iyy>0.00275062</iyy>
-          <iyz>0</iyz>
-          <izz>0.00008316</izz>
-	</inertia>
+        <pose>0 0 0 0 0 0</pose>
+        <mass>0.31</mass>
+        <inertia>
+                <ixx>0.00279048</ixx>
+                <ixy>0</ixy>
+                <ixz>-0.00003956</ixz>
+                <iyy>0.00275062</iyy>
+                <iyz>0</iyz>
+                <izz>0.00008316</izz>
+        </inertia>
       </inertial>
       <collision name="leg_bar_${prefix}_bar_collision">
-	<geometry>
+      <geometry>
           <cylinder>
             <length>${bar_length}</length>
             <radius>${bar_radius}</radius>
           </cylinder>
-	</geometry>
-	<max_contacts>10</max_contacts>
-	<surface>
-          <contact>
-            <ode/>
-          </contact>
-          <bounce/>
-          <friction>
-            <ode/>
-          </friction>
-	</surface>
+      </geometry>
+      <max_contacts>10</max_contacts>
       </collision>
       <visual name="rover_amalia_leg_bar_${prefix}_bar_visual">
-	<pose>0 0 0 0 0 0</pose>
-	<geometry>
-          <cylinder>
-            <length>${bar_length}</length>
-            <radius>${bar_radius}</radius>
-          </cylinder>
-	</geometry>
+        <pose>0 ${-0.018*reflect_xz} 0 0 0 ${-pi/2 + pi/2*reflect_xz}</pose>
+      <geometry>
+        <mesh>
+          <uri>model://${model_root}/meshes/leg.dae</uri>
+        </mesh>
+      </geometry>
       </visual>
     </link>
     <link name="rover_amalia_leg_wheel_${prefix}">
-      <pose>${Ox*reflect_yz} ${(Oy+wheel_length/2+bar_radius+0.001)*reflect_xz} ${Oz + wheel_radius} 0 0 0</pose>
+      <pose>${Ox*reflect_yz} ${(Oy+wheel_length/2+bar_radius+0.01)*reflect_xz} ${Oz + wheel_radius} 0 0 0</pose>
       <inertial>
-	<pose>0 0 0 0 0 0</pose>
-	<mass>1.1</mass>
-	<inertia>
-	  <ixx>0.00222713</ixx>
-	  <iyy>0.00353418</iyy>
-	  <izz>0.00222499</izz>
-	  <ixy>0</ixy>
-	  <ixz>0</ixz>
-	  <iyz>0</iyz>
-	</inertia>
+        <pose>0 0 0 0 0 0</pose>
+        <mass>1.1</mass>
+        <inertia>
+          <ixx>0.00222713</ixx>
+          <iyy>0.00353418</iyy>
+          <izz>0.00222499</izz>
+          <ixy>0</ixy>
+          <ixz>0</ixz>
+          <iyz>0</iyz>
+        </inertia>
       </inertial>
       <collision name="rover_amalia_leg_wheel_${prefix}_collision">
-	<pose>0 0 0 ${pi/2} 0 0</pose>
-	<geometry>
-          <cylinder>
-            <length>${wheel_length}</length>
-            <radius>${wheel_radius}</radius>
-          </cylinder>
-	</geometry>
-	<max_contacts>10</max_contacts>
+      <pose>0 0 0 ${pi/2} 0 0</pose>
+      <geometry>
+              <cylinder>
+                <length>${wheel_length}</length>
+                <radius>${wheel_radius}</radius>
+              </cylinder>
+      </geometry>
+      <max_contacts>10</max_contacts>
       </collision>
       <visual name="rover_amalia_leg_wheel_${prefix}_visual">
-	<pose>0 0 0 0 0 0</pose>
-	<geometry>
+        <pose>0 0 0 0 0 ${-pi/2 + pi/2*reflect_xz}</pose>
+        <geometry>
           <mesh>
             <uri>model://${model_root}/meshes/wheel.dae</uri>
           </mesh>
-	</geometry>
+        </geometry>
       </visual>
       <self_collide>0</self_collide>

File: definitions/rover_amalia_turret/rover_amalia_turret.xacro (robot description, xacro)
@@ -17,4 +17,5 @@
       <size>0.09 0.03 0.05 </size>
   </xacro:property>
+  <xacro:property name="rover_amalia_turret_cam_baseline" value="0.18"/>
   <xacro:property name="rover_amalia_turret_pan_tilt_height" value="0.04"/>
   <xacro:property name="rover_amalia_turret_tilt_hinge_pose">
@@ -55,5 +56,5 @@
       <xacro:insert_block name="rover_amalia_turret_tilt_base_pose"/>
       <visual name="rover_amalia_turret_tilt_base_visual">
-        <pose>-0.016 -0.02 0.015 0 0 0</pose>
+        <pose>-0.020 -0.025 0.015 0 0 0</pose>
         <geometry>
           <mesh>
@@ -63,5 +64,5 @@
       </visual>
       <collision name="rover_amalia_turret_tilt_base_collision">
-        <pose>-0.02 0 0.01 0 0 0</pose>
+        <pose>-0.02 -0.025 0.01 0 0 0</pose>
         <xacro:insert_block name="rover_amalia_turret_tilt_hinge_pose"/>
         <geometry>
@@ -93,13 +94,4 @@
         </geometry>
         <max_contacts>10</max_contacts>
-        <surface>
-          <contact>
-            <ode/>
-          </contact>
-          <bounce/>
-          <friction>
-            <ode/>
-          </friction>
-        </surface>
       </collision>
       <visual name="rover_amalia_turret_tilt_hinge_visual">
@@ -111,14 +103,46 @@
         </geometry>
       </visual>
-      <visual name="rover_amalia_turret_camera_set_visual">
-        <pose>0 0 0.052 0 0 0</pose>
-        <geometry>
-          <mesh>
-            <uri>model://rover_amalia_turret/meshes/pantilt_payload.dae</uri>
-          </mesh>
-        </geometry>
-      </visual>
+      <visual name="rover_amalia_turret_camera_left_visual">
+        <pose>0 ${-rover_amalia_turret_cam_baseline/2} 0.0525 0 0 0</pose>
+        <geometry>
+          <mesh>
+            <uri>model://rover_amalia_turret/meshes/camera.dae</uri>
+          </mesh>
+        </geometry>
+      </visual>
+      <visual name="rover_amalia_turret_tof_visual">
+        <pose>0 0 0.080 0 0 0</pose>
+        <geometry>
+          <mesh>
+            <uri>model://rover_amalia_turret/meshes/tof.dae</uri>
+          </mesh>
+        </geometry>
+      </visual>
+      <visual name="rover_amalia_turret_camera_right_visual">
+        <pose>0 ${rover_amalia_turret_cam_baseline/2} 0.0525 0 0 0</pose>
+        <geometry>
+          <mesh>
+            <uri>model://rover_amalia_turret/meshes/camera.dae</uri>
+          </mesh>
+        </geometry>
+      </visual>
+      <visual name="rover_amalia_turret_camera_base">
+        <pose>0 0 0.04 0 0 0</pose>
+        <geometry>
+          <box>
+            <size>0.02 0.205 0.001</size>
+          </box>
+        </geometry>
+      </visual>
+      <collision name="rover_amalia_turret_payload_collision">
+        <pose>0 0 0.08 0 0 0</pose>
+        <geometry>
+          <box>
+            <size>0.07 0.205 0.09</size>
+          </box>
+        </geometry>
+      </collision>
       <sensor name="depth_camera" type="depth">
-        <pose>0 0 0 0 0 0</pose>
+        <pose>0 0 0.080 0 0 0</pose>
         <camera>
           <horizontal_fov>0.767944</horizontal_fov>
@@ -129,6 +153,6 @@
           </image>
           <clip>
-            <near>0.8</near>
-            <far>9</far>
+            <near>0.05</near>
+            <far>5</far>
           </clip>
         </camera>
@@ -158,6 +182,7 @@
         <update_rate>60</update_rate>
         <visualize>true</visualize>
+        <!--warning: the left and right are inverted, but it is ok -->
         <camera name="left">
-          <pose>0 0 0 0 0 0</pose>
+          <pose>0 ${rover_amalia_turret_cam_baseline/2} 0.0525 0 0 0</pose>
           <horizontal_fov>1.047</horizontal_fov>
           <image>
@@ -166,10 +191,10 @@
           </image>
           <clip>
-            <near>0.4</near>
+            <near>0.05</near>
             <far>100</far>
           </clip>
         </camera>
         <camera name="right">
-          <pose>0 0 0 0 0 0</pose>
+          <pose>0 ${-rover_amalia_turret_cam_baseline/2} 0.0525 0 0 0</pose>
           <horizontal_fov>1.047</horizontal_fov>
           <image>
@@ -178,5 +203,5 @@
           </image>
           <clip>
-            <near>0.4</near>
+            <near>0.05</near>
             <far>100</far>
           </clip>
@@ -190,5 +215,5 @@
           <frameName>left_camera_optical_frame</frameName>
           <rightFrameName>right_camera_optical_frame</rightFrameName>
-          <hackBaseline>0.07</hackBaseline>
+          <hackBaseline>${rover_amalia_turret_cam_baseline}</hackBaseline>
           <distortionK1>0.0</distortionK1>
           <distortionK2>0.0</distortionK2>

File: definitions/rover_amalia_turret_inertials/rover_amalia_turret_inertials.xacro (robot description, xacro)
@@ -61,5 +61,5 @@
         <geometry>
           <box>
-            <size>0.05 0.05 0.05</size>
+            <size>0.05 0.05 0.005</size>
           </box>
         </geometry>
