Commit message: Imported mass, inertia tensor from Adams
The accurate values for the mass and the inertia tensor for chassis,
wheels, and suspension shafts have been imported from the Adams
simulation to the respective .xacro files.

File: definitions/rover_amalia_chassis/rover_amalia_chassis.xacro (robot description, xacro)
@@ -1,17 +1,17 @@
-<?xml version="1.0" ?>
-<robot name="rover_amalia_chassis" xmlns:xacro="http://www.ros.org/wiki/xacro">
-  <xacro:property name="pi" value="3.1415926"/>
+<?xml version="1.0" encoding="utf-8"?>
+<robot name="rover_amalia_chassis" xmlns:xacro="http://www.w3.org/2001/XMLSchema-instance">
+  <xacro:property name="pi" value="3.1415926" />
   <xacro:property name="rover_amalia_chassis_turret_base_size">
-     <size>0.089 0.064 0.046</size>
+    <size>0.089 0.064 0.046</size>
   </xacro:property>
   <xacro:property name="rover_amalia_chassis_body_size">
-     <!--<size>0.492 0.334 0.1</size>-->
-     <size>${body_size_x} ${body_size_y} ${body_size_z}</size>
+    <!--<size>0.492 0.334 0.1</size>-->
+    <size>${body_size_x} ${body_size_y} ${body_size_z}</size>
   </xacro:property>
-  <xacro:property name="rover_amalia_chassis_rangefinder_size_y" value="0.01"/>
+  <xacro:property name="rover_amalia_chassis_rangefinder_size_y" value="0.01" />
   <xacro:property name="rover_amalia_chassis_rangefinder_size">
     <size>${rover_amalia_chassis_rangefinder_size_y} 0.03 ${rover_amalia_chassis_rangefinder_size_y}</size>
   </xacro:property>
-  <xacro:property name="rover_amalia_chassis_turret_base_z" value="0.073"/>
+  <xacro:property name="rover_amalia_chassis_turret_base_z" value="0.073" />
   <xacro:macro name="rover_amalia_chassis" params="Ox Oy Oz body_size_x body_size_y body_size_z turret_base_x turret_base_y">
     <link name="rover_amalia_chassis">
@@ -19,13 +19,13 @@
       <inertial>
         <pose>0.0216667 0 -0.0215556 0 -0 0</pose>
-        <mass>30</mass>
-        <!--<inertia>-->
-          <!--<ixx>900.12</ixx>-->
-          <!--<ixy>-3.46945e-18</ixy>-->
-          <!--<ixz>-0.0139533</ixz>-->
-          <!--<iyy>900.352</iyy>-->
-          <!--<iyz>0</iyz>-->
-          <!--<izz>900.455</izz>-->
-        <!--</inertia>-->
+        <mass>15.6</mass>
+        <inertia>
+          <ixx>0.6385976</ixx>
+          <ixy>0</ixy>
+          <ixz>0</ixz>
+          <iyy>0.521</iyy>
+          <iyz>0</iyz>
+          <izz>0.318954</izz>
+        </inertia>
       </inertial>
       <visual name="rover_amalia_chassis_body_visual">
@@ -41,5 +41,5 @@
         <geometry>
           <box>
-            <xacro:insert_block name="rover_amalia_chassis_body_size"/>
+            <xacro:insert_block name="rover_amalia_chassis_body_size" />
           </box>
         </geometry>
@@ -50,5 +50,5 @@
         <geometry>
           <box>
-            <xacro:insert_block name="rover_amalia_chassis_turret_base_size"/>
+            <xacro:insert_block name="rover_amalia_chassis_turret_base_size" />
           </box>
         </geometry>
@@ -59,5 +59,5 @@
         <geometry>
           <box>
-            <xacro:insert_block name="rover_amalia_chassis_turret_base_size"/>
+            <xacro:insert_block name="rover_amalia_chassis_turret_base_size" />
           </box>
         </geometry>
@@ -67,5 +67,5 @@
         <geometry>
           <box>
-            <xacro:insert_block name="rover_amalia_chassis_rangefinder_size"/>
+            <xacro:insert_block name="rover_amalia_chassis_rangefinder_size" />
           </box>
         </geometry>
@@ -75,5 +75,5 @@
         <geometry>
           <box>
-            <xacro:insert_block name="rover_amalia_chassis_rangefinder_size"/>
+            <xacro:insert_block name="rover_amalia_chassis_rangefinder_size" />
           </box>
         </geometry>
@@ -83,5 +83,5 @@
         <geometry>
           <box>
-            <xacro:insert_block name="rover_amalia_chassis_rangefinder_size"/>
+            <xacro:insert_block name="rover_amalia_chassis_rangefinder_size" />
           </box>
         </geometry>
@@ -91,5 +91,5 @@
         <geometry>
           <box>
-            <xacro:insert_block name="rover_amalia_chassis_rangefinder_size"/>
+            <xacro:insert_block name="rover_amalia_chassis_rangefinder_size" />
           </box>
         </geometry>

File: definitions/rover_amalia_leg/rover_amalia_leg.xacro (robot description, xacro)
@@ -6,80 +6,92 @@
     <link name="rover_amalia_leg_bar_${prefix}">
       <pose>${Ox*reflect_yz} ${Oy*reflect_xz} ${Oz+rover_amalia_leg_bar_z} 0 0 0</pose>
-    <collision name="leg_bar_${prefix}_bar_collision">
-      <geometry>
-        <cylinder>
-          <length>${bar_length}</length>
-          <radius>${bar_radius}</radius>
-        </cylinder>
-      </geometry>
-      <max_contacts>10</max_contacts>
-      <surface>
-        <contact>
-          <ode/>
-        </contact>
-        <bounce/>
-        <friction>
-          <ode/>
-        </friction>
-      </surface>
-    </collision>
-    <visual name="rover_amalia_leg_bar_${prefix}_bar_visual">
-      <pose>0 0 0 0 0 0</pose>
-      <geometry>
-        <cylinder>
-          <length>${bar_length}</length>
-          <radius>${bar_radius}</radius>
-        </cylinder>
-      </geometry>
-    </visual>
-  </link>
-  <link name="rover_amalia_leg_wheel_${prefix}">
-    <pose>${Ox*reflect_yz} ${(Oy+wheel_length/2+bar_radius+0.001)*reflect_xz} ${Oz + wheel_radius} 0 0 0</pose>
-    <inertial>
-      <pose>0 0 0 0 0 0</pose>
-      <mass>5</mass>
-      <inertia>
-        <ixx>100</ixx>
-        <ixy>0</ixy>
-        <ixz>0</ixz>
-        <iyy>100</iyy>
-        <iyz>0</iyz>
-        <izz>100</izz>
-      </inertia>
-    </inertial>
-    <collision name="rover_amalia_leg_wheel_${prefix}_collision">
-      <pose>0 0 0 ${pi/2} 0 0</pose>
-      <geometry>
-        <cylinder>
-          <length>${wheel_length}</length>
-          <radius>${wheel_radius}</radius>
-        </cylinder>
-      </geometry>
-      <max_contacts>10</max_contacts>
-    </collision>
-    <visual name="rover_amalia_leg_wheel_${prefix}_visual">
-      <pose>0 0 0 0 0 0</pose>
-      <geometry>
-        <mesh>
-          <uri>model://${model_root}/meshes/wheel.dae</uri>
-        </mesh>
-      </geometry>
-    </visual>
-    <self_collide>0</self_collide>
-    <kinematic>0</kinematic>
-    <gravity>1</gravity>
-  </link>
-  <joint name="rover_amalia_leg_shaft_${prefix}" type="revolute">
-    <child>rover_amalia_leg_wheel_${prefix}</child>
-    <parent>rover_amalia_leg_bar_${prefix}</parent>
-    <axis>
-      <xyz>0 1 0</xyz>
-      <limit>
-        <lower>-1e+16</lower>
-        <upper>1e+16</upper>
-      </limit>
-      <use_parent_model_frame>1</use_parent_model_frame>
-    </axis>
-  </joint>
+      <inertial>
+	<pose>0 0 0 0 0 0</pose>
+	<mass>0.31</mass>
+	<inertia>
+          <ixx>0.00279048</ixx>
+          <ixy>0</ixy>
+          <ixz>-0.00003956</ixz>
+          <iyy>0.00275062</iyy>
+          <iyz>0</iyz>
+          <izz>0.00008316</izz>
+	</inertia>
+      </inertial>
+      <collision name="leg_bar_${prefix}_bar_collision">
+	<geometry>
+          <cylinder>
+            <length>${bar_length}</length>
+            <radius>${bar_radius}</radius>
+          </cylinder>
+	</geometry>
+	<max_contacts>10</max_contacts>
+	<surface>
+          <contact>
+            <ode/>
+          </contact>
+          <bounce/>
+          <friction>
+            <ode/>
+          </friction>
+	</surface>
+      </collision>
+      <visual name="rover_amalia_leg_bar_${prefix}_bar_visual">
+	<pose>0 0 0 0 0 0</pose>
+	<geometry>
+          <cylinder>
+            <length>${bar_length}</length>
+            <radius>${bar_radius}</radius>
+          </cylinder>
+	</geometry>
+      </visual>
+    </link>
+    <link name="rover_amalia_leg_wheel_${prefix}">
+      <pose>${Ox*reflect_yz} ${(Oy+wheel_length/2+bar_radius+0.001)*reflect_xz} ${Oz + wheel_radius} 0 0 0</pose>
+      <inertial>
+	<pose>0 0 0 0 0 0</pose>
+	<mass>1.1</mass>
+	<inertia>
+	  <ixx>0.00353418</ixx>
+	  <iyy>0.00222499</iyy>
+	  <izz>0.00222713</izz>
+	  <ixy>0</ixy>
+	  <izx>0</izx>
+	  <iyz>0</iyz>
+	</inertia>
+      </inertial>
+      <collision name="rover_amalia_leg_wheel_${prefix}_collision">
+	<pose>0 0 0 ${pi/2} 0 0</pose>
+	<geometry>
+          <cylinder>
+            <length>${wheel_length}</length>
+            <radius>${wheel_radius}</radius>
+          </cylinder>
+	</geometry>
+	<max_contacts>10</max_contacts>
+      </collision>
+      <visual name="rover_amalia_leg_wheel_${prefix}_visual">
+	<pose>0 0 0 0 0 0</pose>
+	<geometry>
+          <mesh>
+            <uri>model://${model_root}/meshes/wheel.dae</uri>
+          </mesh>
+	</geometry>
+      </visual>
+      <self_collide>0</self_collide>
+      <kinematic>0</kinematic>
+      <gravity>1</gravity>
+    </link>
+    <joint name="rover_amalia_leg_shaft_${prefix}" type="revolute">
+      <child>rover_amalia_leg_wheel_${prefix}</child>
+      <parent>rover_amalia_leg_bar_${prefix}</parent>
+      <axis>
+	<xyz>0 1 0</xyz>
+	<limit>
+          <lower>-1e+16</lower>
+          <upper>1e+16</upper>
+	</limit>
+	<use_parent_model_frame>1</use_parent_model_frame>
+      </axis>
+    </joint>
   </xacro:macro>
 </robot>

Commit message: add materials

File: definitions/rover_amalia_chassis/rover_amalia_chassis.xacro (robot description, xacro)
@@ -37,4 +37,8 @@
           </mesh>
         </geometry>
+        <material>
+          <diffuse>0.4 0.4 0.4 1</diffuse>
+          <specular>1 1 1 1</specular>
+        </material>
       </visual>
       <collision name="rover_amalia_chassis_body_collision">
@@ -63,4 +67,8 @@
           </box>
         </geometry>
+        <material>
+          <diffuse>0.4 0.4 0.4 1</diffuse>
+          <specular>1 1 1 1</specular>
+        </material>
       </visual>
       <visual name="rover_amalia_chassis_cpci">
@@ -71,4 +79,8 @@
           </mesh>
         </geometry>
+        <material>
+          <diffuse>0.4 0.4 0.4 1</diffuse>
+          <specular>1 1 1 1</specular>
+        </material>
       </visual>
       <visual name="rover_amalia_chassis_front_up_rangefinder_visual">
@@ -79,4 +91,8 @@
           </box>
         </geometry>
+        <material>
+          <ambient>0.1 0.1 0.1 1</ambient>
+          <diffuse>0 0 0 1</diffuse>
+        </material>
       </visual>
       <visual name="rover_amalia_chassis_front_down_rangefinder_visual">
@@ -87,4 +103,8 @@
           </box>
         </geometry>
+        <material>
+          <ambient>0.1 0.1 0.1 1</ambient>
+          <diffuse>0 0 0 1</diffuse>
+        </material>
       </visual>
       <sensor name="range_front_down_ray" type="ray">
@@ -123,4 +143,8 @@
           </box>
         </geometry>
+        <material>
+          <diffuse>0 0 0 1</diffuse>
+          <!--<specular>0.1 0.1 0.1 0.1</specular>-->
+        </material>
       </visual>
       <visual name="rover_amalia_chassis_rear_down_rangefinder_visual">
@@ -131,4 +155,8 @@
           </box>
         </geometry>
+        <material>
+          <ambient>0.1 0.1 0.1 1</ambient>
+          <diffuse>0 0 0 1</diffuse>
+        </material>
       </visual>
       <sensor name="range_rear_down_ray" type="ray">

File: definitions/rover_amalia_leg/rover_amalia_leg.xacro (robot description, xacro)
@@ -64,7 +64,25 @@
         <geometry>
           <mesh>
-            <uri>model://${model_root}/meshes/wheel.dae</uri>
+            <uri>model://${model_root}/meshes/motor.dae</uri>
           </mesh>
         </geometry>
+        <material>
+          <ambient>1 0.647 0 1</ambient>
+          <diffuse>1 0.647 0 1</diffuse>
+          <specular>1 1 1 0.6</specular>
+        </material>
+      </visual>
+      <visual name="rover_amalia_leg_wheel_${prefix}_visual">
+        <pose>0 0 0 0 0 ${-pi/2 + pi/2*reflect_xz}</pose>
+        <geometry>
+          <mesh>
+            <uri>model://${model_root}/meshes/tire.dae</uri>
+          </mesh>
+        </geometry>
+        <material>
+          <ambient>0.1 0.1 0.1 1</ambient>
+          <diffuse>0 0 0 1</diffuse>
+          <specular>1 1 1 1</specular>
+        </material>
       </visual>
       <self_collide>0</self_collide>

File: definitions/rover_amalia_turret/rover_amalia_turret.xacro (robot description, xacro)
@@ -42,7 +42,24 @@
         <geometry>
           <mesh>
-            <uri>model://rover_amalia_turret/meshes/turret-and-pan-base.dae</uri>
-          </mesh>
-        </geometry>
+            <uri>model://rover_amalia_turret/meshes/turret.dae</uri>
+          </mesh>
+        </geometry>
+        <material>
+          <diffuse>0.4 0.4 0.4 1</diffuse>
+          <specular>1 1 1 1</specular>
+        </material>
+      </visual>
+      <visual name="rover_amalia_turret_bar_pan_base_visual">
+        <pose>-0.012 -0.007 ${bar_height+0.015} 0 0 0</pose>
+        <geometry>
+          <mesh>
+            <uri>model://rover_amalia_turret/meshes/pan_base.dae</uri>
+          </mesh>
+        </geometry>
+        <material>
+          <ambient>0.3 0.3 0.3 1</ambient>
+          <diffuse>0.1 0.1 0.1 1</diffuse>
+          <specular>1 1 1 1</specular>
+        </material>
       </visual>
       <self_collide>0</self_collide>
@@ -62,4 +79,9 @@
           </mesh>
         </geometry>
+        <material>
+          <ambient>0.3 0.3 0.3 1</ambient>
+          <diffuse>0.1 0.1 0.1 1</diffuse>
+          <specular>1 1 1 1</specular>
+        </material>
       </visual>
       <collision name="rover_amalia_turret_tilt_base_collision">
@@ -102,4 +124,9 @@
           </mesh>
         </geometry>
+        <material>
+          <ambient>0.3 0.3 0.3 1</ambient>
+          <diffuse>0.1 0.1 0.1 1</diffuse>
+          <specular>1 1 1 1</specular>
+        </material>
       </visual>
       <visual name="rover_amalia_turret_camera_left_visual">
@@ -110,4 +137,9 @@
           </mesh>
         </geometry>
+        <material>
+          <ambient>0.2 0.2 0.2 1</ambient>
+          <diffuse>0.1 0.1 0.1 1</diffuse>
+          <specular>1 1 1 1</specular>
+        </material>
       </visual>
       <visual name="rover_amalia_turret_tof_visual">
@@ -118,4 +150,9 @@
           </mesh>
         </geometry>
+        <material>
+          <ambient>0.2 0.2 0.2 1</ambient>
+          <diffuse>0.1 0.1 0.1 1</diffuse>
+          <specular>1 1 1 1</specular>
+        </material>
       </visual>
       <visual name="rover_amalia_turret_camera_right_visual">
@@ -126,4 +163,9 @@
           </mesh>
         </geometry>
+        <material>
+          <ambient>0.2 0.2 0.2 1</ambient>
+          <diffuse>0.1 0.1 0.1 1</diffuse>
+          <specular>1 1 1 1</specular>
+        </material>
       </visual>
       <visual name="rover_amalia_turret_camera_base">

Commit message: add imu

File: definitions/rover_amalia_chassis/rover_amalia_chassis.xacro (robot description, xacro)
@@ -14,5 +14,5 @@
   </xacro:property>
   <xacro:property name="rover_amalia_chassis_turret_base_z" value="0.12" />
-  <xacro:property name="rover_amalia_range_finder_z" value="-0.1" />
+  <xacro:property name="rover_amalia_range_finder_z" value="${Oz-0.1}" />
   <xacro:macro name="rover_amalia_chassis" params="Ox Oy Oz body_size_x body_size_y body_size_z turret_base_x turret_base_y">
     <link name="rover_amalia_chassis">
@@ -84,4 +84,9 @@
         </material>
       </visual>
+      <self_collide>0</self_collide>
+      <kinematic>0</kinematic>
+      <gravity>1</gravity>
+    </link>
+    <link name="rover_amalia_rangefinder_front">
       <visual name="rover_amalia_chassis_front_up_rangefinder_visual">
         <pose>0.246 0 ${rover_amalia_range_finder_z} 0 -0 0</pose>
@@ -130,5 +135,5 @@
               <updateRate>20</updateRate>
               <topicName>/ADC/range_front_down</topicName>
-              <frameName>base_link</frameName>
+              <frameName>rover_amalia_rangefinder_front</frameName>
           </plugin>
           <always_on>true</always_on>
@@ -136,4 +141,6 @@
           <visualize>true</visualize>
       </sensor>
+  </link>
+  <link name="rover_amalia_rangefinder_rear">
       <visual name="rover_amalia_chassis_rear_up_rangefinder_visual">
         <pose>-0.246 0 ${rover_amalia_range_finder_z} 3.14159 0.00159265 3.14159</pose>
@@ -144,6 +151,6 @@
         </geometry>
         <material>
-          <diffuse>0 0 0 1</diffuse>
-          <!--<specular>0.1 0.1 0.1 0.1</specular>-->
+          <ambient>0.1 0.1 0.1 1</ambient>
+          <diffuse>0 0 0 1</diffuse>
         </material>
       </visual>
@@ -182,5 +189,5 @@
               <updateRate>20</updateRate>
               <topicName>/ADC/range_rear_down</topicName>
-              <frameName>base_link</frameName>
+              <frameName>rover_amalia_rangefinder_rear</frameName>
           </plugin>
           <always_on>true</always_on>
@@ -188,8 +195,51 @@
           <visualize>true</visualize>
       </sensor>
-      <self_collide>0</self_collide>
-      <kinematic>0</kinematic>
-      <gravity>1</gravity>
-    </link>
+  </link>
+  <joint name="rover_amalia_joint_chassis_rangefinder_front" type="revolute">
+    <child>rover_amalia_rangefinder_front</child>
+    <parent>rover_amalia_chassis</parent>
+    <axis>
+      <xyz>0 0 1</xyz>
+      <limit>
+        <lower>-1e-16</lower>
+        <upper>1e-16</upper>
+        <effort>1000</effort>
+        <velocity>1000</velocity>
+      </limit>
+    </axis>
+  </joint>
+  <joint name="rover_amalia_joint_chassis_rangefinder_rear" type="revolute">
+    <child>rover_amalia_rangefinder_rear</child>
+    <parent>rover_amalia_chassis</parent>
+    <axis>
+      <xyz>0 0 1</xyz>
+      <limit>
+        <lower>-1e-16</lower>
+        <upper>1e-16</upper>
+        <effort>1000</effort>
+        <velocity>1000</velocity>
+      </limit>
+    </axis>
+  </joint>
+  <plugin filename="libgazebo_ros_joint_state_publisher.so" name="rangefinder_rear_p">
+    <robotNamespace></robotNamespace>
+    <jointName>rover_amalia_joint_chassis_rangefinder_rear</jointName>
+    <updateRate>10</updateRate>
+  </plugin>
+  <plugin filename="libgazebo_ros_joint_state_publisher.so" name="rangefinder_front_p">
+    <robotNamespace></robotNamespace>
+    <jointName>rover_amalia_joint_chassis_rangefinder_front</jointName>
+    <updateRate>10</updateRate>
+  </plugin>
+  <plugin name="imu_plugin" filename="libgazebo_ros_imu.so">
+    <alwaysOn>true</alwaysOn>
+    <bodyName>rover_amalia_chassis</bodyName>
+    <topicName>imu_data</topicName>
+    <serviceName>imu_service</serviceName>
+    <gaussianNoise>0.0</gaussianNoise>
+    <updateRate>10.0</updateRate>
+    <xyzOffset>0 0 0</xyzOffset>
+    <rpyOffset>0 0 0</rpyOffset>
+  </plugin>
   </xacro:macro>
 </robot>

File: definitions/rover_amalia_turret/rover_amalia_turret.xacro (robot description, xacro)
@@ -209,5 +209,5 @@
           <cameraInfoTopicName>camera_info</cameraInfoTopicName>
           <cameraName>depth_cam</cameraName>
-          <frameName>/base_link</frameName>
+          <frameName>/rover_amalia_turret_tilt_hinge</frameName>
           <pointCloudCutoff>0.001</pointCloudCutoff>
           <distortionK1>0.0</distortionK1>
@@ -255,6 +255,7 @@
           <imageTopicName>image_raw</imageTopicName>
           <cameraInfoTopicName>camera_info</cameraInfoTopicName>
-          <frameName>left_camera_optical_frame</frameName>
-          <rightFrameName>right_camera_optical_frame</rightFrameName>
+          <!--TODO: change this, add two frames-->
+          <frameName>/rover_amalia_turret_tilt_hinge</frameName>
+          <rightFrameName>/rover_amalia_turret_tilt_hinge</rightFrameName>
           <hackBaseline>${rover_amalia_turret_cam_baseline}</hackBaseline>
           <distortionK1>0.0</distortionK1>
