Commit message: add camera_set_visual

File: definitions/rover_amalia_turret/rover_amalia_turret.xacro (robot description, xacro)
@@ -128,14 +128,14 @@
         </geometry>
       </visual>
-      <!--<visual name="braccio_visual_camera">-->
-        <!--<pose>1.59519e-05 3.18404e-05 -0.06 1.57159 0.00159265 -1.57159</pose>-->
-        <!--<geometry>-->
-          <!--<box>-->
-            <!--<size>0.2 0.04 0.04</size>-->
-          <!--</box>-->
-        <!--</geometry>-->
-      <!--</visual>-->
+      <visual name="rover_amalia_turret_camera_set_visual">
+        <pose>0 0 0.03 0 0 0</pose>
+        <geometry>
+          <box>
+            <size>0.02 0.08 0.02</size>
+          </box>
+        </geometry>
+      </visual>
       <sensor name="depth_camera" type="depth">
-        <pose>0.0 0.0 0.0 0.0 3.14 0.0</pose>
+        <pose>0 0 0 0 ${pi} 0</pose>
         <camera>
           <horizontal_fov>1.578</horizontal_fov>

Commit message: mass, inertia tensor of turret set to better temporary values

File: definitions/rover_amalia_turret/rover_amalia_turret.xacro (robot description, xacro)
@@ -17,5 +17,5 @@
     <pose>${Ox} ${Oy-0.01} ${Oz+bar_height+rover_amalia_turret_pan_base_height+rover_amalia_turret_pan_tilt_height/2} 0 0 0</pose>
   </xacro:property>
-  <xacro:property name="rover_amalia_turret_tilt_base_size">
+  <xacrop:roperty name="rover_amalia_turret_tilt_base_size">
     <size>0.06 0.02 ${rover_amalia_turret_pan_tilt_height}</size>
   </xacro:property>
@@ -26,12 +26,12 @@
       <inertial>
         <pose>0 0 0 0 0 0</pose>
-        <mass>1</mass>
+        <mass>0.5</mass>
         <inertia>
-          <ixx>100</ixx>
+          <ixx>0.001</ixx>
           <ixy>0</ixy>
           <ixz>0</ixz>
-          <iyy>100</iyy>
+          <iyy>0.001</iyy>
           <iyz>0</iyz>
-          <izz>100</izz>
+          <izz>0.001</izz>
         </inertia>
       </inertial>
@@ -64,10 +64,10 @@
         <mass>1</mass>
         <inertia>
-          <ixx>100</ixx>
+          <ixx>0.001</ixx>
           <ixy>0</ixy>
           <ixz>0</ixz>
-          <iyy>100</iyy>
+          <iyy>0.00100</iyy>
           <iyz>0</iyz>
-          <izz>100</izz>
+          <izz>0.00100</izz>
         </inertia>
       </inertial>
@@ -94,10 +94,10 @@
         <mass>2</mass>
         <inertia>
-          <ixx>200.001</ixx>
+          <ixx>0.00200001</ixx>
           <ixy>0</ixy>
           <ixz>0</ixz>
-          <iyy>200.001</iyy>
+          <iyy>0.00200001</iyy>
           <iyz>0</iyz>
-          <izz>200</izz>
+          <izz>0.00200</izz>
         </inertia>
       </inertial>

Commit message: fix typo

File: definitions/rover_amalia_turret/rover_amalia_turret.xacro (robot description, xacro)
@@ -17,5 +17,5 @@
     <pose>${Ox} ${Oy-0.01} ${Oz+bar_height+rover_amalia_turret_pan_base_height+rover_amalia_turret_pan_tilt_height/2} 0 0 0</pose>
   </xacro:property>
-  <xacrop:roperty name="rover_amalia_turret_tilt_base_size">
+  <xacro:property name="rover_amalia_turret_tilt_base_size">
     <size>0.06 0.02 ${rover_amalia_turret_pan_tilt_height}</size>
   </xacro:property>

Commit message: fix pantilt mesh

File: definitions/rover_amalia_turret/rover_amalia_turret.xacro (robot description, xacro)
@@ -7,6 +7,7 @@
   </xacro:property>
   <xacro:property name="rover_amalia_turret_tilt_base_height" value="0.02"/>
+  <xacro:property name="pan_base_height" value="0.043"/>
   <xacro:property name="rover_amalia_turret_tilt_base_pose">
-    <pose>${Ox} ${Oy} ${Oz+bar_height+rover_amalia_turret_tilt_base_height/2} 0 0 0</pose>
+    <pose>${Ox} ${Oy+0.015} ${Oz+pan_base_height+bar_height+rover_amalia_turret_tilt_base_height/2} 0 0 0</pose>
   </xacro:property>
   <xacro:property name="rover_amalia_turret_tilt_base_size">
@@ -15,5 +16,5 @@
   <xacro:property name="rover_amalia_turret_pan_tilt_height" value="0.04"/>
   <xacro:property name="rover_amalia_turret_tilt_hinge_pose">
-    <pose>${Ox} ${Oy-0.01} ${Oz+bar_height+rover_amalia_turret_tilt_base_height+rover_amalia_turret_pan_tilt_height/2} 0 0 0</pose>
+    <pose>${Ox} ${Oy-0.01} ${Oz+pan_base_height+bar_height+rover_amalia_turret_tilt_base_height+rover_amalia_turret_pan_tilt_height/2} 0 0 0</pose>
   </xacro:property>
   <xacro:property name="rover_amalia_turret_tilt_hinge_size">
@@ -48,8 +49,7 @@
         <pose>0 0 ${bar_height/2} 0 0 0</pose>
         <geometry>
-          <cylinder>
-            <length>${bar_height}</length>
-            <radius>${rover_amalia_turret_bar_radius}</radius>
-          </cylinder>
+          <mesh>
+            <uri>model://rover_amalia_turret/meshes/turret-and-pan-base.dae</uri>
+          </mesh>
         </geometry>
       </visual>

Commit message: fix turret inertials

File: definitions/rover_amalia_turret/rover_amalia_turret.xacro (robot description, xacro)
@@ -8,4 +8,7 @@
   <xacro:property name="rover_amalia_turret_tilt_base_height" value="0.02"/>
   <xacro:property name="pan_base_height" value="0.043"/>
+  <xacro:property name="rover_amalia_turret_pan_base_pose">
+    <pose>${Ox} ${Oy+0.015} ${Oz+pan_base_height+bar_height+rover_amalia_turret_tilt_base_height/2}-0.01 0 0 0</pose>
+  </xacro:property>
   <xacro:property name="rover_amalia_turret_tilt_base_pose">
     <pose>${Ox} ${Oy+0.015} ${Oz+pan_base_height+bar_height+rover_amalia_turret_tilt_base_height/2} 0 0 0</pose>
@@ -23,18 +26,21 @@
   <xacro:property name="rover_amalia_turret_robot_namespace" value="rover_amalia" />
   <xacro:macro name="rover_amalia_turret" params="Ox Oy Oz bar_height">
+    <link name="rover_amalia_turret_bar_inertial_dummy">
+      <xacro:insert_block name="rover_amalia_turret_bar_pose"/>
+      <inertial>
+        <pose>0 0 0 0 0 0</pose>
+        <mass>0.78</mass>
+        <inertia>
+          <ixx>0.00000027555</ixx>
+          <ixy>0</ixy>
+          <ixz>0</ixz>
+          <iyy>0.00000027555</iyy>
+          <iyz>0</iyz>
+          <izz>0.00000027755</izz>
+        </inertia>
+      </inertial>
+    </link>
     <link name="rover_amalia_turret_bar">
       <xacro:insert_block name="rover_amalia_turret_bar_pose"/>
-      <!--<inertial>-->
-        <!--<pose>0 0 0 0 0 0</pose>-->
-        <!--<mass>0.78</mass>-->
-        <!--<inertia>-->
-          <!--<ixx>0.00000027555</ixx>-->
-          <!--<ixy>0</ixy>-->
-          <!--<ixz>0</ixz>-->
-          <!--<iyy>0.00000027555</iyy>-->
-          <!--<iyz>0</iyz>-->
-          <!--<izz>0.00000027755</izz>-->
-        <!--</inertia>-->
-      <!--</inertial>-->
       <collision name="rover_amalia_turret_bar_collision">
         <pose>0 0 ${bar_height/2} 0 0 0</pose>
@@ -58,33 +64,36 @@
       <gravity>1</gravity>
     </link>
+    <link name="rover_amalia_turret_pan_base_inertial_dummy">
+      <xacro:insert_block name="rover_amalia_turret_pan_base_pose"/>
+      <inertial>
+        <pose>-0.00699 0.17952 0.02755 0 0 0</pose>
+        <mass>0.22386</mass>
+        <inertia>
+          <ixx>0.00010575745</ixx>
+          <ixy>0.00002524815</ixy>
+          <ixz>0</ixz>
+          <iyy>0.00100</iyy>
+          <iyz>0</iyz>
+          <izz>0.00021796864</izz>
+        </inertia>
+      </inertial>
+    </link>
+    <link name="rover_amalia_turret_tilt_base_inertial_dummy">
+      <inertial>
+        <pose>0.012 -0.21853 0.02754  0 0 0</pose>
+        <pose>0 0 0 0 0 0</pose>
+        <mass>0.02786</mass>
+        <inertia>
+          <ixx>0.00002247622</ixx>
+          <ixy>0.</ixy>
+          <ixz>0</ixz>
+          <iyy>0.00001850151</iyy>
+          <iyz>0</iyz>
+          <izz>0.00000707185</izz>
+        </inertia>
+      </inertial>
+    </link>
     <link name="rover_amalia_turret_tilt_base">
       <xacro:insert_block name="rover_amalia_turret_tilt_base_pose"/>
-      <!--correct inertial for pan base, use later-->
-      <!--<inertial>-->
-        <!--<pose>-0.00699 0.17952 0.02755 0 0 0</pose>-->
-        <!--<mass>0.22386</mass>-->
-        <!--<inertia>-->
-          <!--<ixx>0.00010575745</ixx>-->
-          <!--<ixy>0.00002524815</ixy>-->
-          <!--<ixz>0</ixz>-->
-          <!--<iyy>0.00100</iyy>-->
-          <!--<iyz>0</iyz>-->
-          <!--<izz>0.00021796864</izz>-->
-        <!--</inertia>-->
-      <!--</inertial>-->
-      <!--this are ok, leave them:-->
-      <!--<inertial>-->
-        <!--<pose>0.012 -0.21853 0.02754  0 0 0</pose>-->
-        <!--<pose>0 0 0 0 0 0</pose>-->
-        <!--<mass>0.02786</mass>-->
-        <!--<inertia>-->
-          <!--<ixx>0.00002247622</ixx>-->
-          <!--<ixy>0.</ixy>-->
-          <!--<ixz>0</ixz>-->
-          <!--<iyy>0.00001850151</iyy>-->
-          <!--<iyz>0</iyz>-->
-          <!--<izz>0.00000707185</izz>-->
-        <!--</inertia>-->
-      <!--</inertial>-->
       <visual name="rover_amalia_turret_tilt_base_visual">
         <pose>-0.016 -0.02 0.015 0 0 0</pose>

Commit message: add depth camera frame

File: definitions/rover_amalia_turret/rover_amalia_turret.xacro (robot description, xacro)
@@ -143,17 +143,4 @@
         </material>
       </visual>
-      <visual name="rover_amalia_turret_tof_visual">
-        <pose>0 0 0.080 0 0 0</pose>
-        <geometry>
-          <mesh>
-            <uri>model://rover_amalia_turret/meshes/tof.dae</uri>
-          </mesh>
-        </geometry>
-        <material>
-          <ambient>0.2 0.2 0.2 1</ambient>
-          <diffuse>0.1 0.1 0.1 1</diffuse>
-          <specular>1 1 1 1</specular>
-        </material>
-      </visual>
       <visual name="rover_amalia_turret_camera_right_visual">
         <pose>0 ${rover_amalia_turret_cam_baseline/2} 0.0525 0 0 0</pose>
@@ -185,39 +172,4 @@
         </geometry>
       </collision>
-      <sensor name="depth_camera" type="depth">
-        <pose>0 0 0.080 0 0 0</pose>
-        <camera>
-          <horizontal_fov>0.767944</horizontal_fov>
-          <image>
-            <width>176</width>
-            <height>144</height>
-            <format>R8G8B8</format>
-          </image>
-          <clip>
-            <near>0.05</near>
-            <far>5</far>
-          </clip>
-        </camera>
-        <plugin filename="libgazebo_ros_depth_camera.so" name="depth_camera_plugin">
-          <alwaysOn>1</alwaysOn>
-          <robotNamespace>${rover_amalia_turret_robot_namespace}</robotNamespace>
-          <updateRate>25.0</updateRate>
-          <imageTopicName>image_raw</imageTopicName>
-          <depthImageTopicName>depth_raw</depthImageTopicName>
-          <depthImageCameraInfoTopicName>camera_info</depthImageCameraInfoTopicName>
-          <pointCloudTopicName>points</pointCloudTopicName>
-          <cameraInfoTopicName>camera_info</cameraInfoTopicName>
-          <cameraName>depth_cam</cameraName>
-          <frameName>/rover_amalia_turret_tilt_hinge</frameName>
-          <pointCloudCutoff>0.001</pointCloudCutoff>
-          <distortionK1>0.0</distortionK1>
-          <distortionK2>0.0</distortionK2>
-          <distortionK3>0.0</distortionK3>
-          <distortionT1>0.0</distortionT1>
-          <distortionT2>0.0</distortionT2>
-        </plugin>
-        <always_on>true</always_on>
-        <update_rate>25.0</update_rate>
-      </sensor>
       <sensor name="camera" type="multicamera">
         <always_on>1</always_on>
@@ -277,4 +229,77 @@
       </inertial>
     </link>
+    <link name="rover_amalia_turret_depth_camera_link">
+      <pose> 0.2 0 0.824 0 0 0</pose>
+      <visual name="rover_amalia_turret_tof_visual">
+        <geometry>
+          <mesh>
+            <uri>model://rover_amalia_turret/meshes/tof.dae</uri>
+          </mesh>
+        </geometry>
+        <material>
+          <ambient>0.2 0.2 0.2 1</ambient>
+          <diffuse>0.1 0.1 0.1 1</diffuse>
+          <specular>1 1 1 1</specular>
+        </material>
+      </visual>
+      <sensor name="depth_camera" type="depth">
+        <camera>
+          <horizontal_fov>0.767944</horizontal_fov>
+          <image>
+            <width>176</width>
+            <height>144</height>
+            <format>R8G8B8</format>
+          </image>
+          <clip>
+            <near>0.05</near>
+            <far>5</far>
+          </clip>
+        </camera>
+        <plugin filename="libgazebo_ros_depth_camera.so" name="depth_camera_plugin">
+          <alwaysOn>1</alwaysOn>
+          <robotNamespace>${rover_amalia_turret_robot_namespace}</robotNamespace>
+          <updateRate>25.0</updateRate>
+          <imageTopicName>image_raw</imageTopicName>
+          <depthImageTopicName>depth_raw</depthImageTopicName>
+          <depthImageCameraInfoTopicName>camera_info</depthImageCameraInfoTopicName>
+          <pointCloudTopicName>points</pointCloudTopicName>
+          <cameraInfoTopicName>camera_info</cameraInfoTopicName>
+          <cameraName>depth_cam</cameraName>
+          <frameName>/rover_amalia_turret_depth_camera_link</frameName>
+          <pointCloudCutoff>0.001</pointCloudCutoff>
+          <distortionK1>0.0</distortionK1>
+          <distortionK2>0.0</distortionK2>
+          <distortionK3>0.0</distortionK3>
+          <distortionT1>0.0</distortionT1>
+          <distortionT2>0.0</distortionT2>
+        </plugin>
+        <always_on>true</always_on>
+        <update_rate>25.0</update_rate>
+      </sensor>
+      <self_collide>0</self_collide>
+      <kinematic>0</kinematic>
+      <gravity>0</gravity>
+      <inertial>
+        <mass>0.000001</mass>
+      </inertial>
+    </link>
+    <joint name="rover_amalia_hinge_depth_camera_link" type="revolute">
+      <child>rover_amalia_turret_depth_camera_link</child>
+      <parent>rover_amalia_turret_tilt_hinge</parent>
+      <axis>
+        <xyz>0 1 0</xyz>
+        <limit>
+          <lower>-1e-16</lower>
+          <upper>1e-16</upper>
+          <effort>1000</effort>
+          <velocity>1000</velocity>
+        </limit>
+      </axis>
+    </joint>
+    <plugin filename="libgazebo_ros_joint_state_publisher.so" name="depth_camera_p">
+      <robotNamespace></robotNamespace>
+      <jointName>rover_amalia_hinge_depth_camera_link</jointName>
+      <updateRate>10</updateRate>
+    </plugin>
     <joint name="rover_amalia_turret_pan" type="revolute">
       <child>rover_amalia_turret_tilt_base</child>
@@ -322,12 +347,14 @@
     </plugin>
     <plugin filename="libgazebo_ros_joint_state_publisher.so" name="pan">
+      <!--keep update rate lower than camera rate-->
       <robotNamespace></robotNamespace>
       <jointName>rover_amalia_turret_pan</jointName>
-      <updateRate>30</updateRate>
+      <updateRate>20</updateRate>
     </plugin>
     <plugin filename="libgazebo_ros_joint_state_publisher.so" name="tilt">
+      <!--keep update rate lower than camera rate-->
       <robotNamespace></robotNamespace>
       <jointName>rover_amalia_turret_tilt</jointName>
-      <updateRate>30</updateRate>
+      <updateRate>20</updateRate>
     </plugin>
   </xacro:macro>
