Commit message: fix leg missing visual

File: definitions/rover_amalia_leg/rover_amalia_leg.xacro (robot description, xacro)
@@ -60,5 +60,5 @@
       <max_contacts>10</max_contacts>
       </collision>
-      <visual name="rover_amalia_leg_wheel_${prefix}_visual">
+      <visual name="rover_amalia_leg_wheel_${prefix}_motor_visual">
         <pose>0 0 0 0 0 ${-pi/2 + pi/2*reflect_xz}</pose>
         <geometry>
@@ -73,5 +73,5 @@
         </material>
       </visual>
-      <visual name="rover_amalia_leg_wheel_${prefix}_visual">
+      <visual name="rover_amalia_leg_wheel_${prefix}_tire_visual">
         <pose>0 0 0 0 0 ${-pi/2 + pi/2*reflect_xz}</pose>
         <geometry>
